File: 4_Layer_Board/percussiveInterface-3.1.kicad_pcb (KiCad board)
At the start: 4 copper layers, 460 x 97.7 mm, 108 parts, among them U1 Teensy4.1, U10 SS39ET, U11 SS39ET, U12 SS39ET, U13 SS39ET, U14 SS39ET, U15 SS39ET, U16 SS39ET, U17 SS39ET, U18 SS39ET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

Commit message: more notes
Routing:
- net +5V: track 416.5 -> 421.3 mm, vias 36 -> 40
