File: percussiveInterface-3.2/percussiveInterface-3.2/magnetometer_array/magnetometer_array.kicad_pcb (KiCad board)
At the start: 4 copper layers, 122.6 x 14 mm, 33 parts, among them J2 Conn_01x21_Pin, U1 SM225-10E, U10 SM225-10E, U11 SM225-10E, U12 SM225-10E, U13 SM225-10E, U14 SM225-10E, U15 SM225-10E, U16 SM225-10E, U2 SM225-10E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

Commit message: slightl<y new
Parts:
- moved C12 0.64 mm to (185.4, 110.8)
Routing:
- net v+: track 32.8 -> 52.7 mm, vias 1 -> 17
- net MISO: track 296.3 -> 299.7 mm
- net SS6: track 12.5 -> 14.4 mm
- net SS3: track 27.8 -> 29.7 mm
- net SS4: track 22.7 -> 24.6 mm
- net SS2: track 32.8 -> 34.7 mm
- net SS1: track 37.9 -> 39.8 mm
- net SS5: track 17.6 -> 19.5 mm
- net SS9: track 9.99 -> 11.9 mm
- added copper zone on In1.Cu, net v+

Commit message: stuff
Parts:
- J2: footprint Connector_PinHeader_2.54mm:PinHeader_1x21_P2.54mm_Horizontal -> Connector_PinHeader_2.54mm:PinHeader_1x21_P2.54mm_Vertical
- moved U8 1.27 mm to (156.2, 111.8)
- moved J2 1.26 mm to (186.7, 107.3)
Routing:
- net MOSI: track 136.8 -> 143.0 mm
- net v+: track 52.7 -> 51.1 mm, vias 17 -> 16
- net SS5: track 19.5 -> 18.2 mm
- net SS4: track 24.6 -> 23.3 mm
- net SS3: track 29.7 -> 28.4 mm
- net SS2: track 34.7 -> 33.5 mm
- net SS1: track 39.8 -> 38.6 mm
- net MISO: track 299.7 -> 300.5 mm
- net SS13: track 32.2 -> 32.8 mm
- added copper zone on In2.Cu, net GND
Other:
- board size 122.6 x 14 mm -> 122.6 x 12.1 mm
