File: percussiveInterface-3.2/percussiveInterface-3.2/percussiveInterface-3.2.kicad_sch (KiCad schematic)
At the start: 133 parts, among them IC1 ADG731BSUZ, IC2 TXU0304PWR, U1 SM225-10E, U10 SM225-10E, U11 SM225-10E, U12 SM225-10E, U13 SM225-10E, U14 SM225-10E, U15 SM225-10E, U16 SM225-10E, U17 SM225-10E, U18 SM225-10E, U19 SM225-10E, U2 SM225-10E, U20 SM225-10E, U21 SM225-10E, U22 SM225-10E, U23 SM225-10E, U24 SM225-10E, U25 SM225-10E, U26 SM225-10E, U27 SM225-10E, U28 SM225-10E, U29 SM225-10E, U3 SM225-10E, U30 SM225-10E, U31 SM225-10E, U32 SM225-10E, U34 ESP32-WROOM-32, U4 SM225-10E, U5 SM225-10E, U6 SM225-10E, U7 SM225-10E, U8 SM225-10E, U9 SM225-10E

Commit message: layout 3.2
Parts:
- added C35, C36: .1µ, Capacitor_SMD:C_0201_0603Metric, symbol Device:C_Small
- added C37: 33µF, symbol Device:C_Polarized
- added C38: .47µF, symbol Device:C_Polarized
- added IC3: LM3940IMP-3.3_NOPB, SOT230P700X180-4N, symbol LM3940IMP-3_3_NOPB:LM3940IMP-3.3_NOPB
- added J1: PRG EN, digikey-footprints:PinHeader_1x2_P2.54mm_Drill1.02mm, symbol dk_Rectangular-Connectors-Headers-Male-Pins:22-23-2021
- added J2: 302-S101, digikey-footprints:PinHeader_2x5_P2.54mm_Drill1.2mm, symbol dk_Rectangular-Connectors-Headers-Male-Pins:302-S101
- C33: footprint (none) -> Capacitor_SMD:CP_Elec_6.3x3
Connections:
- net CS0: now also J2.6
- net CS1 unbuffered: now also J2.8
- net at IC2.1 (VCCA): now also IC2.14 (VCCB), C35.1
- net OE: now reaches IC2.8 (OE)
- net OE: now also U34.28 (IO17)
- net LED SDO: now reaches D1.4 (SDI)
- net LED SDO: now also U34.31 (IO19)
- net LED CLK: now reaches D1.5 (CKI)
- net LED CLK: now also U34.30 (IO18)
- net at U34.2 (VDD): now also C36.1
- net at U34.25 (IO0): now also J1.1
- net UART0 RX: now reaches U34.34 (RXD0/IO3)
- net UART0 RX: now also J2.4
- net UART0 TX: now reaches U34.35 (TXD0/IO1)
- net UART0 TX: now also J2.2
- new net: C37.2, C38.2, IC3.4 (GND_2)
- new net: C36.2, J1.2
Other:
- note added: "APA102 RGB LED Array"
- note added: "Magnetometer Array"
- note added: "SPI Buffer"
- note added: "SPI MULTIPLEXER"
- title: (none) -> Rotor Platine
- moved on the sheet: C1, C10, C11, C12, C13, C14, C15, C16, C17, C18, C19, C2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

Commit message: nochmal update
Parts:
- added C39: .1µ, Capacitor_SMD:C_0201_0603Metric, symbol Device:C_Small
- added IC4: DRV5021A1QDBZT, SOT95P237X112-3N, symbol DRV5021A1QDBZT:DRV5021A1QDBZT
- added R1: 10k, symbol Device:R
Connections:
- net at U34.29 (IO5): now also IC4.2 (OUT), R1.2
- new net: C39.1, IC4.1 (VCC)
- new net: C39.2, IC4.3 (GND)
Other:
- moved on the sheet: J2

Commit message: updates
Parts:
- removed C39: .1µ, Capacitor_SMD:C_0201_0603Metric, symbol Device:C_Small
- removed D17, D18, D19, D20, D21, D22, D23, D24, D33, D34, D35, D36, D37, D38, D39, D40, D41, D42, D43, D44, D45, D46, D47, D48, D49, D50, D51, D52, D53, D54, D55, D56, D57, D58, D59, D60, D61, D62, D63, D64: APA102-2020, LED_SMD:LED-APA102-2020, symbol LED:APA102-2020
- removed IC4: DRV5021A1QDBZT, SOT95P237X112-3N, symbol DRV5021A1QDBZT:DRV5021A1QDBZT
- added IC10, IC11, IC12, IC13, IC14, IC15, IC16, IC17, IC18, IC19, IC20, IC21, IC22, IC23, IC24, IC25, IC26, IC27, IC28, IC29, IC30, IC31, IC32, IC33, IC34, IC35, IC36, IC37, IC38, IC39, IC4, IC40, IC41, IC42, IC43, IC44, IC45, IC46, IC47, IC48, IC49, IC5, IC50, IC51, IC52, IC53, IC54, IC55, IC56, IC57, IC58, IC59, IC6, IC60, IC61, IC62, IC63, IC64, IC65, IC66, IC67, IC68, IC69, IC7, IC70, IC71, IC72, IC73, IC74, IC75, IC76, IC77, IC78, IC79, IC8, IC80, IC81, IC82, IC83, IC84, IC85, IC86, IC87, IC88, IC89, IC9, IC90, IC91: VCNL4040M3OE, VCNL4040M3OE, symbol VCNL4040M3OE:VCNL4040M3OE
- added R2: 10K, symbol Device:R
- added U33: MPU-6050, Sensor_Motion:InvenSense_QFN-24_4x4mm_P0.5mm, symbol Sensor_Motion:MPU-6050
- added U35: QRE1113GR, OptoDevice:OnSemi_CASE100CY, symbol Sensor_Proximity:QRE1113GR
- C37, C38: symbol Device:C_Polarized -> Device:C
- R1: value 10k -> 100
Connections:
- net at D25.4 (SDI): now also D16.3 (SDO)
- net at D25.5 (CKI): now also D16.2 (CKO)
- net at U34.29 (IO5): now also R2.1, U35.3; no longer R1.2
- new net: IC32.1 (GND), IC33.1 (GND)
- new net: IC32.2 (K(SENSOR)), IC33.2 (K(SENSOR))
- new net: IC32.3 (VDD), IC33.3 (VDD)
- new net: IC32.4 (A), IC33.4 (A)
- new net: IC32.5 (K(LED)), IC33.5 (K(LED))
- new net: IC32.6 (INT), IC33.6 (INT)
- new net: IC32.7 (SDAT), IC33.7 (SDAT)
- new net: IC32.8 (SCLK), IC33.8 (SCLK)
- new net: IC72.1 (GND), IC73.1 (GND)
- new net: IC72.2 (K(SENSOR)), IC73.2 (K(SENSOR))
- new net: IC72.3 (VDD), IC73.3 (VDD)
- new net: IC72.4 (A), IC73.4 (A)
- new net: IC72.5 (K(LED)), IC73.5 (K(LED))
- new net: IC72.6 (INT), IC73.6 (INT)
- new net: IC72.7 (SDAT), IC73.7 (SDAT)
- new net: IC72.8 (SCLK), IC73.8 (SCLK)
- new net: IC83.1 (GND), IC84.1 (GND)
- new net: IC83.2 (K(SENSOR)), IC84.2 (K(SENSOR))
- new net: IC83.3 (VDD), IC84.3 (VDD)
- new net: IC83.4 (A), IC84.4 (A)
- new net: IC83.5 (K(LED)), IC84.5 (K(LED))
- new net: IC83.6 (INT), IC84.6 (INT)
- new net: IC83.7 (SDAT), IC84.7 (SDAT)
- new net: IC83.8 (SCLK), IC84.8 (SCLK)
- new net: IC87.1 (GND), IC88.1 (GND)
- new net: IC87.2 (K(SENSOR)), IC88.2 (K(SENSOR))
- new net: IC87.3 (VDD), IC88.3 (VDD)
- new net: IC87.4 (A), IC88.4 (A)
- new net: IC87.5 (K(LED)), IC88.5 (K(LED))
- new net: IC87.6 (INT), IC88.6 (INT)
- new net: IC87.7 (SDAT), IC88.7 (SDAT)
- new net: IC87.8 (SCLK), IC88.8 (SCLK)
- new net: IC35.1 (GND), IC36.1 (GND)
- new net: IC35.2 (K(SENSOR)), IC36.2 (K(SENSOR))
- new net: IC35.3 (VDD), IC36.3 (VDD)
- new net: IC35.4 (A), IC36.4 (A)
- new net: IC35.5 (K(LED)), IC36.5 (K(LED))
- new net: IC35.6 (INT), IC36.6 (INT)
- new net: IC35.7 (SDAT), IC36.7 (SDAT)
- new net: IC35.8 (SCLK), IC36.8 (SCLK)
- new net: IC21.1 (GND), IC22.1 (GND)
- new net: IC21.2 (K(SENSOR)), IC22.2 (K(SENSOR))
- new net: IC21.3 (VDD), IC22.3 (VDD)
- new net: IC21.4 (A), IC22.4 (A)
- new net: IC21.5 (K(LED)), IC22.5 (K(LED))
- new net: IC21.6 (INT), IC22.6 (INT)
- new net: IC21.7 (SDAT), IC22.7 (SDAT)
- new net: IC21.8 (SCLK), IC22.8 (SCLK)
- new net: IC61.1 (GND), IC62.1 (GND)
- new net: IC61.2 (K(SENSOR)), IC62.2 (K(SENSOR))
- new net: IC61.3 (VDD), IC62.3 (VDD)
- new net: IC61.4 (A), IC62.4 (A)
- new net: IC61.5 (K(LED)), IC62.5 (K(LED))
- new net: IC61.6 (INT), IC62.6 (INT)
- new net: IC61.7 (SDAT), IC62.7 (SDAT)
- new net: IC61.8 (SCLK), IC62.8 (SCLK)
- new net: IC65.1 (GND), IC66.1 (GND)
- new net: IC65.2 (K(SENSOR)), IC66.2 (K(SENSOR))
- new net: IC65.3 (VDD), IC66.3 (VDD)
- new net: IC65.4 (A), IC66.4 (A)
- new net: IC65.5 (K(LED)), IC66.5 (K(LED))
- new net: IC65.6 (INT), IC66.6 (INT)
- new net: IC65.7 (SDAT), IC66.7 (SDAT)
- new net: IC65.8 (SCLK), IC66.8 (SCLK)
- new net: IC79.1 (GND), IC80.1 (GND)
- new net: IC79.2 (K(SENSOR)), IC80.2 (K(SENSOR))
- new net: IC79.3 (VDD), IC80.3 (VDD)
- new net: IC79.4 (A), IC80.4 (A)
- new net: IC79.5 (K(LED)), IC80.5 (K(LED))
- new net: IC79.6 (INT), IC80.6 (INT)
- new net: IC79.7 (SDAT), IC80.7 (SDAT)
- new net: IC79.8 (SCLK), IC80.8 (SCLK)
- new net: IC17.1 (GND), IC18.1 (GND)
- new net: IC17.2 (K(SENSOR)), IC18.2 (K(SENSOR))
- new net: IC17.3 (VDD), IC18.3 (VDD)
- new net: IC17.4 (A), IC18.4 (A)
- new net: IC17.5 (K(LED)), IC18.5 (K(LED))
- new net: IC17.6 (INT), IC18.6 (INT)
- new net: IC17.7 (SDAT), IC18.7 (SDAT)
- new net: IC17.8 (SCLK), IC18.8 (SCLK)
- new net: IC50.1 (GND), IC51.1 (GND)
- new net: IC50.2 (K(SENSOR)), IC51.2 (K(SENSOR))
- new net: IC50.3 (VDD), IC51.3 (VDD)
- new net: IC50.4 (A), IC51.4 (A)
- new net: IC50.5 (K(LED)), IC51.5 (K(LED))
- new net: IC50.6 (INT), IC51.6 (INT)
- new net: IC50.7 (SDAT), IC51.7 (SDAT)
- new net: IC50.8 (SCLK), IC51.8 (SCLK)
- new net: IC28.1 (GND), IC29.1 (GND)
- new net: IC28.2 (K(SENSOR)), IC29.2 (K(SENSOR))
- new net: IC28.3 (VDD), IC29.3 (VDD)
- new net: IC28.4 (A), IC29.4 (A)
- new net: IC28.5 (K(LED)), IC29.5 (K(LED))
- new net: IC28.6 (INT), IC29.6 (INT)
- new net: IC28.7 (SDAT), IC29.7 (SDAT)
- new net: IC28.8 (SCLK), IC29.8 (SCLK)
- new net: IC13.1 (GND), IC14.1 (GND)
- new net: IC13.2 (K(SENSOR)), IC14.2 (K(SENSOR))
- new net: IC13.3 (VDD), IC14.3 (VDD)
- new net: IC13.4 (A), IC14.4 (A)
- new net: IC13.5 (K(LED)), IC14.5 (K(LED))
- new net: IC13.6 (INT), IC14.6 (INT)
- new net: IC13.7 (SDAT), IC14.7 (SDAT)
- new net: IC13.8 (SCLK), IC14.8 (SCLK)
- new net: IC43.1 (GND), IC44.1 (GND)
- new net: IC43.2 (K(SENSOR)), IC44.2 (K(SENSOR))
- new net: IC43.3 (VDD), IC44.3 (VDD)
- new net: IC43.4 (A), IC44.4 (A)
- new net: IC43.5 (K(LED)), IC44.5 (K(LED))
- new net: IC43.6 (INT), IC44.6 (INT)
- new net: IC43.7 (SDAT), IC44.7 (SDAT)
- new net: IC43.8 (SCLK), IC44.8 (SCLK)
- new net: IC6.1 (GND), IC7.1 (GND)
- new net: IC6.2 (K(SENSOR)), IC7.2 (K(SENSOR))
- new net: IC6.3 (VDD), IC7.3 (VDD)
- new net: IC6.4 (A), IC7.4 (A)
- new net: IC6.5 (K(LED)), IC7.5 (K(LED))
- new net: IC6.6 (INT), IC7.6 (INT)
- new net: IC6.7 (SDAT), IC7.7 (SDAT)
- new net: IC6.8 (SCLK), IC7.8 (SCLK)
- new net: IC10.1 (GND), IC11.1 (GND)
- new net: IC10.2 (K(SENSOR)), IC11.2 (K(SENSOR))
- new net: IC10.3 (VDD), IC11.3 (VDD)
- new net: IC10.4 (A), IC11.4 (A)
- new net: IC10.5 (K(LED)), IC11.5 (K(LED))
- new net: IC10.6 (INT), IC11.6 (INT)
- new net: IC10.7 (SDAT), IC11.7 (SDAT)
- new net: IC10.8 (SCLK), IC11.8 (SCLK)
- new net: IC57.1 (GND), IC58.1 (GND)
- new net: IC57.2 (K(SENSOR)), IC58.2 (K(SENSOR))
- new net: IC57.3 (VDD), IC58.3 (VDD)
- new net: IC57.4 (A), IC58.4 (A)
- new net: IC57.5 (K(LED)), IC58.5 (K(LED))
- new net: IC57.6 (INT), IC58.6 (INT)
- new net: IC57.7 (SDAT), IC58.7 (SDAT)
- new net: IC57.8 (SCLK), IC58.8 (SCLK)
- new net: R1.2, U35.1 (A)
- new net: IC24.1 (GND), IC25.1 (GND)
- new net: IC24.2 (K(SENSOR)), IC25.2 (K(SENSOR))
- new net: IC24.3 (VDD), IC25.3 (VDD)
- new net: IC24.4 (A), IC25.4 (A)
- new net: IC24.5 (K(LED)), IC25.5 (K(LED))
- new net: IC24.6 (INT), IC25.6 (INT)
- new net: IC24.7 (SDAT), IC25.7 (SDAT)
- new net: IC24.8 (SCLK), IC25.8 (SCLK)
- new net: IC90.1 (GND), IC91.1 (GND)
- new net: IC90.2 (K(SENSOR)), IC91.2 (K(SENSOR))
- new net: IC90.3 (VDD), IC91.3 (VDD)
- new net: IC90.4 (A), IC91.4 (A)
- new net: IC90.5 (K(LED)), IC91.5 (K(LED))
- new net: IC90.6 (INT), IC91.6 (INT)
- new net: IC90.7 (SDAT), IC91.7 (SDAT)
- new net: IC90.8 (SCLK), IC91.8 (SCLK)
- new net: IC39.1 (GND), IC40.1 (GND)
- new net: IC39.2 (K(SENSOR)), IC40.2 (K(SENSOR))
- new net: IC39.3 (VDD), IC40.3 (VDD)
- new net: IC39.4 (A), IC40.4 (A)
- new net: IC39.5 (K(LED)), IC40.5 (K(LED))
- new net: IC39.6 (INT), IC40.6 (INT)
- new net: IC39.7 (SDAT), IC40.7 (SDAT)
- new net: IC39.8 (SCLK), IC40.8 (SCLK)
- new net: IC46.1 (GND), IC47.1 (GND)
- new net: IC46.2 (K(SENSOR)), IC47.2 (K(SENSOR))
- new net: IC46.3 (VDD), IC47.3 (VDD)
- new net: IC46.4 (A), IC47.4 (A)
- new net: IC46.5 (K(LED)), IC47.5 (K(LED))
- new net: IC46.6 (INT), IC47.6 (INT)
- new net: IC46.7 (SDAT), IC47.7 (SDAT)
- new net: IC46.8 (SCLK), IC47.8 (SCLK)
- new net: IC76.1 (GND), IC77.1 (GND)
- new net: IC76.2 (K(SENSOR)), IC77.2 (K(SENSOR))
- new net: IC76.3 (VDD), IC77.3 (VDD)
- new net: IC76.4 (A), IC77.4 (A)
- new net: IC76.5 (K(LED)), IC77.5 (K(LED))
- new net: IC76.6 (INT), IC77.6 (INT)
- new net: IC76.7 (SDAT), IC77.7 (SDAT)
- new net: IC76.8 (SCLK), IC77.8 (SCLK)
- new net: IC54.1 (GND), IC55.1 (GND)
- new net: IC54.2 (K(SENSOR)), IC55.2 (K(SENSOR))
- new net: IC54.3 (VDD), IC55.3 (VDD)
- new net: IC54.4 (A), IC55.4 (A)
- new net: IC54.5 (K(LED)), IC55.5 (K(LED))
- new net: IC54.6 (INT), IC55.6 (INT)
- new net: IC54.7 (SDAT), IC55.7 (SDAT)
- new net: IC54.8 (SCLK), IC55.8 (SCLK)
- new net: IC68.1 (GND), IC69.1 (GND)
- new net: IC68.2 (K(SENSOR)), IC69.2 (K(SENSOR))
- new net: IC68.3 (VDD), IC69.3 (VDD)
- new net: IC68.4 (A), IC69.4 (A)
- new net: IC68.5 (K(LED)), IC69.5 (K(LED))
- new net: IC68.6 (INT), IC69.6 (INT)
- new net: IC68.7 (SDAT), IC69.7 (SDAT)
- new net: IC68.8 (SCLK), IC69.8 (SCLK)
Other:
- note added: "3,3V REGULATOR"
- note added: "REFLECTIVE RPM METER"
- note added: "use int. pullup"
- moved on the sheet: C1, C10, C11, C12, C13, C14, C15, C16, C17, C18, C19, C2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

Commit message: new arrray
Parts:
- removed C1, C10, C11, C12, C13, C14, C15, C16, C17, C18, C19, C2, C20, C21, C22, C23, C24, C25, C26, C27, C28, C29, C3, C30, C31, C32, C4, C5, C6, C7, C8, C9: 1µ, Capacitor_SMD:C_0201_0603Metric, symbol Device:C_Small
- removed IC10, IC11, IC12, IC13, IC14, IC15, IC16, IC17, IC18, IC19, IC20, IC21, IC22, IC23, IC24, IC25, IC26, IC27, IC28, IC29, IC30, IC31, IC32, IC33, IC34, IC35, IC36, IC37, IC38, IC39, IC4, IC40, IC41, IC42, IC43, IC44, IC45, IC46, IC47, IC48, IC49, IC5, IC50, IC51, IC52, IC53, IC54, IC55, IC56, IC57, IC58, IC59, IC6, IC60, IC61, IC62, IC63, IC64, IC65, IC66, IC67, IC68, IC69, IC7, IC70, IC71, IC72, IC73, IC74, IC75, IC76, IC77, IC78, IC79, IC8, IC80, IC81, IC82, IC83, IC84, IC85, IC86, IC87, IC88, IC89, IC9, IC90, IC91: VCNL4040M3OE, VCNL4040M3OE, symbol VCNL4040M3OE:VCNL4040M3OE
- removed U1, U10, U11, U12, U13, U14, U15, U16, U17, U18, U19, U2, U20, U21, U22, U23, U24, U25, U26, U27, U28, U29, U3, U30, U31, U32, U4, U5, U6, U7, U8, U9: SM225-10E, SON65P250X250X80-7N, symbol SM225-10E:SM225-10E
Other:
- note removed: "Magnetometer Array"
