File: percussiveInterface-3.2/percussiveInterface-3.2/magnetometer_array_2/magnetometer_array_2.kicad_sch (KiCad schematic)
At the start: 69 parts, among them J1 Conn_01x05_Socket, J2 Conn_01x08_Socket, J3 Conn_01x08_Socket, J4 Conn_01x08_Socket, J5 Conn_01x08_Socket, U1 SM225-10E, U10 SM225-10E, U11 SM225-10E, U12 SM225-10E, U13 SM225-10E, U14 SM225-10E, U15 SM225-10E, U16 SM225-10E, U17 SM225-10E, U18 SM225-10E, U19 SM225-10E, U2 SM225-10E, U20 SM225-10E, U21 SM225-10E, U22 SM225-10E, U23 SM225-10E, U24 SM225-10E, U25 SM225-10E, U26 SM225-10E, U27 SM225-10E, U28 SM225-10E, U29 SM225-10E, U3 SM225-10E, U30 SM225-10E, U31 SM225-10E, U32 SM225-10E, U4 SM225-10E, U5 SM225-10E, U6 SM225-10E, U7 SM225-10E, U8 SM225-10E, U9 SM225-10E

Commit message: new magnetoarray
Parts:
- removed C25, C26, C27, C28, C29, C30, C31, C32: C_Small, Capacitor_SMD:C_0201_0603Metric, symbol Device:C_Small
- removed J5: Conn_01x08_Socket, Connector_PinSocket_2.54mm:PinSocket_1x08_P2.54mm_Horizontal, symbol Connector:Conn_01x12_Socket
- removed U25, U26, U27, U28, U29, U30, U31, U32: SM225-10E, NVE:SON65P250X250X80-7N, symbol SM225-10E:SM225-10E
- J1: footprint Connector_PinSocket_2.54mm:PinSocket_1x05_P2.54mm_Horizontal -> Connector_PinSocket_2.54mm:PinSocket_1x05_P2.54mm_Vertical_SMD_Pin1Left
- J2, J3, J4: value Conn_01x08_Socket -> Conn_01x12_Socket; footprint Connector_PinSocket_2.54mm:PinSocket_1x08_P2.54mm_Horizontal -> Connector_PinSocket_2.54mm:PinSocket_1x12_P2.54mm_Vertical_SMD_Pin1Left
Connections:
- net SS25 is gone; now on net SS7: U7.1 (SS)
- net SS26 is gone; now on net SS15: U15.1 (SS)
- net SS27 is gone; now on net SS23: U23.1 (SS)
- net SS29 is gone; now on net SS8: U8.1 (SS)
- net SS30 is gone; now on net SS16: U16.1 (SS)
- net SS31 is gone; now on net SS24: U24.1 (SS)
- net SS10: now also U10.1 (SS); no longer U11.1 (SS)
- net SS11: now also U11.1 (SS); no longer U19.1 (SS)
- net SS12: now also U12.1 (SS)
- net SS13: now also U13.1 (SS); no longer U4.1 (SS)
- net SS14: now also U14.1 (SS); no longer U12.1 (SS)
- net SS15: no longer U20.1 (SS)
- net SS17: now also U17.1 (SS); no longer U5.1 (SS)
- net SS18: now also U18.1 (SS); no longer U13.1 (SS)
- net SS19: now also U19.1 (SS); no longer U21.1 (SS)
- net SS2: now also U2.1 (SS); no longer U9.1 (SS)
- net SS20: now also U20.1 (SS)
- net SS21: now also U21.1 (SS); no longer U6.1 (SS)
- net SS22: now also U22.1 (SS); no longer U14.1 (SS)
- net SS23: no longer U22.1 (SS)
- net SS3: now also U3.1 (SS); no longer U17.1 (SS)
- net SS4: now also U4.1 (SS)
- net SS5: now also U5.1 (SS); no longer U2.1 (SS)
- net SS6: now also U6.1 (SS); no longer U10.1 (SS)
- net SS7: no longer U18.1 (SS)
- net SS9: now also U9.1 (SS); no longer U3.1 (SS)

Commit message: new arrray
Parts:
- J1: footprint Connector_PinSocket_2.54mm:PinSocket_1x05_P2.54mm_Vertical_SMD_Pin1Left -> Connector_Harwin:Harwin_M20-89005xx_1x05_P2.54mm_Horizontal
- J2, J3, J4: footprint Connector_PinSocket_2.54mm:PinSocket_1x12_P2.54mm_Vertical_SMD_Pin1Left -> Connector_Harwin:Harwin_M20-89012xx_1x12_P2.54mm_Horizontal
Changed lines of the file:
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@@
       (effects (font (size 1.27 1.27)) (justify left))
     )
-    (property "Footprint" "Connector_PinSocket_2.54mm:PinSocket_1x12_P2.54mm_Vertical_SMD_Pin1Left" (at 302.26 80.01 0)
+    (property "Footprint" "Connector_Harwin:Harwin_M20-89012xx_1x12_P2.54mm_Horizontal" (at 302.26 80.01 0)
       (effects (font (size 1.27 1.27)) hide)
     )
@@
       (effects (font (size 1.27 1.27)) (justify left))
     )
-    (property "Footprint" "Connector_PinSocket_2.54mm:PinSocket_1x12_P2.54mm_Vertical_SMD_Pin1Left" (at 302.26 151.13 0)
+    (property "Footprint" "Connector_Harwin:Harwin_M20-89012xx_1x12_P2.54mm_Horizontal" (at 302.26 151.13 0)
       (effects (font (size 1.27 1.27)) hide)
     )
@@
       (effects (font (size 1.27 1.27)) (justify left))
     )
-    (property "Footprint" "Connector_PinSocket_2.54mm:PinSocket_1x12_P2.54mm_Vertical_SMD_Pin1Left" (at 302.26 116.84 0)
+    (property "Footprint" "Connector_Harwin:Harwin_M20-89012xx_1x12_P2.54mm_Horizontal" (at 302.26 116.84 0)
       (effects (font (size 1.27 1.27)) hide)
     )
@@
       (effects (font (size 1.27 1.27)) (justify left))
     )
-    (property "Footprint" "Connector_PinSocket_2.54mm:PinSocket_1x05_P2.54mm_Vertical_SMD_Pin1Left" (at 302.26 57.15 0)
-      (effects (font (size 1.27 1.27)) hide)
-    )
+    (property "Footprint" "Connector_Harwin:Harwin_M20-89005xx_1x05_P2.54mm_Horizontal" (at 302.26 57.15 0)
+      (effects (font (size 1.27 1.27)) hide)
+    )
