File: percussiveInterface-3.2/magnetometer_array_2/magnetometer_array_2.kicad_pcb (KiCad board)
At the start: 4 copper layers, 167 x 16 mm, 52 parts, among them J1 Conn_01x05_Socket, J2 Conn_01x12_Socket, J3 Conn_01x12_Socket, J4 Conn_01x12_Socket, U1 SM225-10E, U10 SM225-10E, U11 SM225-10E, U12 SM225-10E, U13 SM225-10E, U14 SM225-10E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

Commit message: many changes
Parts:
- J1: footprint Connector_Harwin:Harwin_M20-89005xx_1x05_P2.54mm_Horizontal -> Connector_PinHeader_2.54mm:PinHeader_1x05_P2.54mm_Horizontal
- J2, J3, J4: footprint Connector_Harwin:Harwin_M20-89012xx_1x12_P2.54mm_Horizontal -> Connector_PinHeader_2.54mm:PinHeader_1x12_P2.54mm_Horizontal
- U1, U10, U11, U12, U13, U14, U15, U16, U17, U18, U19, U2, U20, U21, U22, U23, U24, U3, U4, U5, U6, U7, U8, U9: footprint NVE:SON65P250X250X80-7N -> Own_Library:NVE SM225 10E
- moved J2 15.0 mm to (92.1, 63.4)
- moved J3 15.0 mm to (148.0, 63.4)
- moved J4 15.0 mm to (203.8, 63.4)
- moved J1 8.46 mm to (54.0, 63.4)
Connections:
- J2 pad 1: SS1 -> SS8
- J2 pad 10: SS7 -> SS2
- J2 pad 12: SS8 -> SS1
- J2 pad 3: SS2 -> SS7
- J2 pad 4: SS3 -> SS6
- J2 pad 6: SS4 -> SS5
- J2 pad 7: SS5 -> SS4
- J2 pad 9: SS6 -> SS3
- J3 pad 1: SS9 -> SS16
- J3 pad 10: SS15 -> SS10
- J3 pad 12: SS16 -> SS9
- J3 pad 3: SS10 -> SS15
- J3 pad 4: SS11 -> SS14
- J3 pad 6: SS12 -> SS13
- J3 pad 7: SS13 -> SS12
- J3 pad 9: SS14 -> SS11
- J4 pad 1: SS17 -> SS24
- J4 pad 10: SS23 -> SS18
- J4 pad 12: SS24 -> SS17
- J4 pad 3: SS18 -> SS23
- J4 pad 4: SS19 -> SS22
- J4 pad 6: SS20 -> SS21
- J4 pad 7: SS21 -> SS20
- J4 pad 9: SS22 -> SS19
Routing:
- net SCLK: track 214.2 -> 215.9 mm
- net GND: track 4.47 -> 5.44 mm
- net MOSI: track 220.4 -> 220.9 mm
- net SS5: track 17.5 -> 17.0 mm
Other:
- board size 167 x 16 mm -> 167 x 16.5 mm

Commit message: almost there but not
Changed lines of the file:
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@@
   (segment (start 182.35 51.155) (end 181.33 51.155) (width 0.3) (layer "F.Cu") (net 1))
   (segment (start 91.35 51.155) (end 90.33 51.155) (width 0.3) (layer "F.Cu") (net 1))
-  (via blind (at 151.13 52.705) (size 0.8) (drill 0.4) (layers "F.Cu" "In2.Cu") (free) (net 1))
-  (via blind (at 81.28 52.705) (size 0.8) (drill 0.4) (layers "F.Cu" "In2.Cu") (free) (net 1))
-  (via blind (at 60.325 52.705) (size 0.8) (drill 0.4) (layers "F.Cu" "In2.Cu") (free) (net 1))
+  (via (at 151.13 52.705) (size 0.8) (drill 0.4) (layers "F.Cu" "B.Cu") (free) (net 1))
+  (via (at 81.28 52.705) (size 0.8) (drill 0.4) (layers "F.Cu" "B.Cu") (free) (net 1))
+  (via (at 60.325 52.705) (size 0.8) (drill 0.4) (layers "F.Cu" "B.Cu") (free) (net 1))
   (via (at 56.769 63.373) (size 1) (drill 0.6) (layers "F.Cu" "B.Cu") (free) (net 1))
-  (via blind (at 88.265 52.705) (size 0.8) (drill 0.4) (layers "F.Cu" "In2.Cu") (free) (net 1))
-  (via blind (at 74.295 52.705) (size 0.8) (drill 0.4) (layers "F.Cu" "In2.Cu") (free) (net 1))
-  (via blind (at 137.16 52.705) (size 0.8) (drill 0.4) (layers "F.Cu" "In2.Cu") (free) (net 1))
-  (via blind (at 158.115 52.705) (size 0.8) (drill 0.4) (layers "F.Cu" "In2.Cu") (free) (net 1))
-  (via blind (at 41 51.75) (size 0.8) (drill 0.4) (layers "F.Cu" "In2.Cu") (free) (net 1))
-  (via blind (at 172.085 52.705) (size 0.8) (drill 0.4) (layers "F.Cu" "In2.Cu") (free) (net 1))
-  (via blind (at 46.228 52.705) (size 0.8) (drill 0.4) (layers "F.Cu" "In2.Cu") (free) (net 1))
-  (via blind (at 109.22 52.705) (size 0.8) (drill 0.4) (layers "F.Cu" "In2.Cu") (free) (net 1))
-  (via blind (at 67.31 52.705) (size 0.8) (drill 0.4) (layers "F.Cu" "In2.Cu") (free) (net 1))
-  (via blind (at 186.055 52.705) (size 0.8) (drill 0.4) (layers "F.Cu" "In2.Cu") (free) (net 1))
-  (via blind (at 179.07 52.705) (size 0.8) (drill 0.4) (layers "F.Cu" "In2.Cu") (free) (net 1))
-  (via blind (at 130.175 52.705) (size 0.8) (drill 0.4) (layers "F.Cu" "In2.Cu") (free) (net 1))
-  (via blind (at 102.235 52.705) (size 0.8) (drill 0.4) (layers "F.Cu" "In2.Cu") (free) (net 1))
-  (via blind (at 53.086 52.705) (size 0.8) (drill 0.4) (layers "F.Cu" "In2.Cu") (free) (net 1))
-  (via blind (at 95.25 52.705) (size 0.8) (drill 0.4) (layers "F.Cu" "In2.Cu") (free) (net 1))
-  (via blind (at 116.205 52.705) (size 0.8) (drill 0.4) (layers "F.Cu" "In2.Cu") (free) (net 1))
-  (via blind (at 144.145 52.705) (size 0.8) (drill 0.4) (layers "F.Cu" "In2.Cu") (free) (net 1))
-  (via blind (at 200.025 52.705) (size 0.8) (drill 0.4) (layers "F.Cu" "In2.Cu") (free) (net 1))
-  (via blind (at 193.04 52.705) (size 0.8) (drill 0.4) (layers "F.Cu" "In2.Cu") (free) (net 1))
-  (via blind (at 123.19 52.705) (size 0.8) (drill 0.4) (layers "F.Cu" "In2.Cu") (free) (net 1))
-  (via blind (at 165.1 52.705) (size 0.8) (drill 0.4) (layers "F.Cu" "In2.Cu") (free) (net 1))
+  (via (at 88.265 52.705) (size 0.8) (drill 0.4) (layers "F.Cu" "B.Cu") (free) (net 1))
+  (via (at 74.295 52.705) (size 0.8) (drill 0.4) (layers "F.Cu" "B.Cu") (free) (net 1))
+  (via (at 137.16 52.705) (size 0.8) (drill 0.4) (layers "F.Cu" "B.Cu") (free) (net 1))
+  (via (at 158.115 52.705) (size 0.8) (drill 0.4) (layers "F.Cu" "B.Cu") (free) (net 1))
+  (via (at 41 51.75) (size 0.8) (drill 0.4) (layers "F.Cu" "B.Cu") (free) (net 1))
+  (via (at 172.085 52.705) (size 0.8) (drill 0.4) (layers "F.Cu" "B.Cu") (free) (net 1))
+  (via (at 46.228 52.705) (size 0.8) (drill 0.4) (layers "F.Cu" "B.Cu") (free) (net 1))
+  (via (at 109.22 52.705) (size 0.8) (drill 0.4) (layers "F.Cu" "B.Cu") (free) (net 1))
+  (via (at 67.31 52.705) (size 0.8) (drill 0.4) (layers "F.Cu" "B.Cu") (free) (net 1))
+  (via (at 186.055 52.705) (size 0.8) (drill 0.4) (layers "F.Cu" "B.Cu") (free) (net 1))
+  (via (at 179.07 52.705) (size 0.8) (drill 0.4) (layers "F.Cu" "B.Cu") (free) (net 1))
+  (via (at 130.175 52.705) (size 0.8) (drill 0.4) (layers "F.Cu" "B.Cu") (free) (net 1))
+  (via (at 102.235 52.705) (size 0.8) (drill 0.4) (layers "F.Cu" "B.Cu") (free) (net 1))
+  (via (at 53.086 52.705) (size 0.8) (drill 0.4) (layers "F.Cu" "B.Cu") (free) (net 1))
+  (via (at 95.25 52.705) (size 0.8) (drill 0.4) (layers "F.Cu" "B.Cu") (free) (net 1))
+  (via (at 116.205 52.705) (size 0.8) (drill 0.4) (layers "F.Cu" "B.Cu") (free) (net 1))
+  (via (at 144.145 52.705) (size 0.8) (drill 0.4) (layers "F.Cu" "B.Cu") (free) (net 1))
+  (via (at 200.025 52.705) (size 0.8) (drill 0.4) (layers "F.Cu" "B.Cu") (free) (net 1))
+  (via (at 193.04 52.705) (size 0.8) (drill 0.4) (layers "F.Cu" "B.Cu") (free) (net 1))
+  (via (at 123.19 52.705) (size 0.8) (drill 0.4) (layers "F.Cu" "B.Cu") (free) (net 1))
+  (via (at 165.1 52.705) (size 0.8) (drill 0.4) (layers "F.Cu" "B.Cu") (free) (net 1))
   (segment (start 53.975 63.373) (end 56.769 63.373) (width 0.8) (layer "B.Cu") (net 1))
   (segment (start 42.164 58.801) (end 41.05 57.687) (width 0.3) (layer "F.Cu") (net 2))
