File: percussiveInterface-3.2/main_board_old/percussiveInterface-3.2.kicad_sch (KiCad schematic)
At the start: 44 parts, among them IC1 ADG731BSUZ, IC2 TXU0304PWR, IC3 LM3940IMP-3.3_NOPB, J1 PRG EN, J2 302-S101, J3 Conn_01x12_Socket, J4 Conn_01x12_Socket, J7 Conn_01x05_Socket, J8 Conn_01x12_Socket, U33 MPU-6050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

Commit message: many changes
Parts:
- removed C33: 100µF, Capacitor_SMD:CP_Elec_6.3x3, symbol Device:C_Polarized_Small
- removed D1, D10, D11, D12, D13, D14, D15, D16, D2, D25, D26, D27, D28, D29, D3, D30, D31, D32, D4, D5, D6, D7, D8, D9: APA102-2020, LED_SMD:LED-APA102-2020, symbol LED:APA102-2020
- removed J3, J4, J8: Conn_01x12_Socket, symbol Own_Symbols:Hirose_MDF7-12S-2.54DSA(55)
- removed J7: Conn_01x05_Socket, symbol Own_Symbols:Hirose_MDF7-05S-2.54DSA(55)
- added J10, J9: SAMTEC-SLW-108-01-X-S, Own_Library:SAMTEC-SLW-108-01-X-S, symbol SAMTEC-SLW-108-01-X-S:SAMTEC-SLW-108-01-X-S
- added J11: Screw_Terminal_01x02, TerminalBlock_Phoenix:TerminalBlock_Phoenix_MKDS-1,5-2-5.08_1x02_P5.08mm_Horizontal, symbol ConnectorZZ:Screw_Terminal_01x02
- added J3: BSW-120-X-X-S, Own_Library:SAMTEC_BSW-120-X-X-S, symbol BSW-120-X-X-S:BSW-120-X-X-S
- added J4: BSW-134-X-X-S, Own_Library:SAMTEC_BSW-134-X-X-S, symbol BSW-134-X-X-S:BSW-134-X-X-S
- added J5, J6, J7, J8: SLW-104-01-G-S, Own_Library:SAMTEC_SLW-104-01-G-S, symbol SLW-104-01-G-S:SLW-104-01-G-S
- C37, C38: footprint (none) -> Capacitor_SMD:C_0402_1005Metric
- IC1: footprint QFP50P900X900X120-48N -> Own_Library:TQFP48
- IC2: footprint SOP65P640X120-14N -> Package_SO:TSSOP-14_4.4x5mm_P0.65mm
- IC3: footprint SOT230P700X180-4N -> Package_TO_SOT_SMD:SOT-223
- R1, R2: footprint (none) -> Resistor_SMD:R_0402_1005Metric
Connections:
- net CS0: no longer J2.6
- net CS1 unbuffered: no longer J2.8
- net CLK: no longer names the net of IC2.12 (B2Y)
- net CLK: no longer IC1.19 (SCLK)
- net CS1: no longer names the net of IC2.11 (B3Y)
- net CS1: no longer IC1.43 (D)
- net MISO: no longer names the net of IC2.10 (B4)
- net MOSI: no longer names the net of IC2.13 (B1Y)
- net MOSI: no longer IC1.18 (DIN)
- net UART0 RX: no longer names the net of J2.4
- net UART0 RX: no longer U34.34 (RXD0/IO3)
- net UART0 TX: no longer names the net of J2.2
- net UART0 TX: no longer U34.35 (TXD0/IO1)
- net muxCS1: no longer names the net of IC1.12 (S1)
- net muxCS10: no longer names the net of IC1.3 (S10)
- net muxCS11: no longer names the net of IC1.2 (S11)
- net muxCS12: no longer names the net of IC1.1 (S12)
- net muxCS13: no longer names the net of IC1.48 (S13)
- net muxCS14: no longer names the net of IC1.47 (S14)
- net muxCS15: no longer names the net of IC1.46 (S15)
- net muxCS16: no longer names the net of IC1.45 (S16)
- net muxCS17: no longer names the net of IC1.25 (S17)
- net muxCS18: no longer names the net of IC1.26 (S18)
- net muxCS19: no longer names the net of IC1.27 (S19)
- net muxCS2: no longer names the net of IC1.11 (S2)
- net muxCS20: no longer names the net of IC1.28 (S20)
- net muxCS21: no longer names the net of IC1.29 (S21)
- net muxCS22: no longer names the net of IC1.30 (S22)
- net muxCS23: no longer names the net of IC1.31 (S23)
- net muxCS24: no longer names the net of IC1.32 (S24)
- net muxCS25: no longer names the net of IC1.33 (S25)
- net muxCS26: no longer names the net of IC1.34 (S26)
- net muxCS27: no longer names the net of IC1.35 (S27)
- net muxCS28: no longer names the net of IC1.36 (S28)
- net muxCS29: no longer names the net of IC1.37 (S29)
- net muxCS3: no longer names the net of IC1.10 (S3)
- net muxCS30: no longer names the net of IC1.38 (S30)
- net muxCS31: no longer names the net of IC1.39 (S31)
- net muxCS32: no longer names the net of IC1.40 (S32)
- net muxCS4: no longer names the net of IC1.9 (S4)
- net muxCS5: no longer names the net of IC1.8 (S5)
- net muxCS6: no longer names the net of IC1.7 (S6)
- net muxCS7: no longer names the net of IC1.6 (S7)
- net muxCS8: no longer names the net of IC1.5 (S8)
- net muxCS9: no longer names the net of IC1.4 (S9)
Other:
- note removed: "APA102 RGB LED Array"
- moved on the sheet: C34, C35, C36, C37, C38, IC1, IC2, IC3, J1, J2, R1, R2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
