File: percussiveInterface-3.2/main_board_old/main_board-3.2.kicad_sch (KiCad schematic)
At the start: 25 parts, among them IC1 ADG731BSUZ, IC2 TXU0304PWR, IC3 LM3940IMP-3.3_NOPB, J1 PRG EN, J10 SAMTEC-SLW-108-01-X-S, J11 Screw_Terminal_01x02, J2 302-S101, J3 BSW-120-X-X-S, J4 BSW-134-X-X-S, J5 SLW-104-01-G-S, J6 SLW-104-01-G-S, J7 SLW-104-01-G-S, J8 SLW-104-01-G-S, J9 SAMTEC-SLW-108-01-X-S, U34 ESP32-WROOM-32, U35 QRE1113GR

Commit message: almost there but not
Parts:
- removed J1: PRG EN, digikey-footprints:PinHeader_1x2_P2.54mm_Drill1.02mm, symbol dk_Rectangular-Connectors-Headers-Male-Pins:22-23-2021
- removed J2: 302-S101, digikey-footprints:PinHeader_2x5_P2.54mm_Drill1.2mm, symbol dk_Rectangular-Connectors-Headers-Male-Pins:302-S101
- removed J4: BSW-134-X-X-S, Own_Library:SAMTEC_BSW-134-X-X-S, symbol BSW-134-X-X-S:BSW-134-X-X-S
- added C1: 22µ, Capacitor_SMD:C_0402_1005Metric, symbol Device:C_Small
- added C2: 1µ, Capacitor_SMD:C_0402_1005Metric, symbol Device:C_Small
- added C3, C4: 22pF, Capacitor_SMD:C_0402_1005Metric, symbol Device:C_Small
- added C5, C6: 0.1µ, Capacitor_SMD:C_0402_1005Metric, symbol Device:C_Small
- added J1: 0022232041, digikey-footprints:PinHeader_1x4_P2.54mm_Drill1.02mm, symbol dk_Rectangular-Connectors-Headers-Male-Pins:0022232041
- added J12, J2: BSW-112-X-X-S, Own_Library:SAMTEC_BSW-112-X-X-S, symbol BSW-112-X-X-S:BSW-112-X-X-S
- added JP1: SolderJumper_2_Bridged, Jumper:SolderJumper-2_P1.3mm_Open_Pad1.0x1.5mm, symbol Jumper:SolderJumper_2_Bridged
- added R3: 10k, Resistor_SMD:R_0402_1005Metric, symbol Device:R
- added SW1: SW_Boot, Button_Switch_SMD:SW_SPST_B3U-1000P, symbol Switch:SW_Push
- added SW2: SW_Reset, Button_Switch_SMD:SW_SPST_B3U-1000P, symbol Switch:SW_Push
- added U1, U2: SN74LV1T34DBV, Package_TO_SOT_SMD:SOT-23-5, symbol Logic_LevelTranslator:SN74LV1T34DBV
- C34, C35, C36: value .1µ -> 0.1µ; footprint Capacitor_SMD:C_0201_0603Metric -> Capacitor_SMD:C_0402_1005Metric
- C38: value .47µF -> 0.47µF
- H1: footprint MountingHole:MountingHole_4.3mm_M4_ISO7380_Pad_TopBottom -> MountingHole:MountingHole_2.2mm_M2_DIN965_Pad
- IC1: footprint Own_Library:TQFP48 -> Package_QFP:TQFP-48_7x7mm_P0.5mm
- J3: value BSW-120-X-X-S -> BSW-120-04-X-S
- U34: value ESP32-WROOM-32 -> ESP32-S3-WROOM-1-n16r8; footprint RF_Module:ESP32-WROOM-32 -> Own_Library:ESP32-S3-WROOM-1-N16R2; symbol RF_Module:ESP32-WROOM-32 -> ESP32-S3-WROOM-1-N16R2:ESP32-S3-WROOM-1-N16R2; Availability (none) -> In Stock; Check_prices (none) -> https://www.snapeda.com/parts/ESP32-S3-WROOM-1-N16R2/Espres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; MANUFACTURER (none) -> Espressif; MAXIMUM_PACKAGE_HEIGHT (none) -> 3.25mm; MF (none) -> Espressif Systems; MP (none) -> ESP32-S3-WROOM-1-N16R8; PARTREV (none) -> v1.0; Package (none) -> NON STANDARD Espressif Systems; Price (none) -> None; Purchase-URL (none) -> https://www.snapeda.com/api/url_track_click_mouser/?unipart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; STANDARD (none) -> Manufacturer Recommendations; SnapEDA_Link (none) -> https://www.snapeda.com/parts/ESP32-S3-WROOM-1-N16R2/Espres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
Connections:
- net 3.3V: now also IC2.8 (OE), J3.05, C1.1, R3.1; no longer D1.1 (VDD), J3.01
- net 5V: now also D1.1 (VDD), C5.2, C6.2, JP1.1 (A), U1.5 (VCC), U2.5 (VCC); no longer C38.1, IC3.1 (IN)
- net CLK: now also J3.04; no longer J3.02
- net CLK unbuffered: now also U34.21 (IO13); no longer U34.13 (IO14)
- net CS0: now also U34.39 (IO1); no longer U34.23 (IO15)
- net CS1 unbuffered: now also U34.20 (IO12); no longer U34.27 (IO16)
- net GND: now also J3.02, U34.41 (GND), C1.2, C2.2, C3.2, C4.2, C5.1, C6.1, J1.4, J12.02, J12.05, J12.08, J12.11, J2.02, J2.05, J2.08, J2.11, SW1.1, SW2.1, U1.3 (GND), U2.3 (GND); no longer J3.04, U34.1 (GND), U34.15 (GND), U34.38 (GND), U34.39 (GND)
- net LDC_CLK: now also U34.10 (IO17); no longer U34.7 (IO35)
- net LDC_CS: now also U34.8 (IO15); no longer U34.5 (SENSOR_VN)
- net LDC_INT: now also U34.9 (IO16); no longer U34.4 (SENSOR_VP)
- net LED CLK: now also D1.2 (CKO), D1.5 (CKI), U1.4 (Y); no longer D1.3 (SDO), D1.4 (SDI), U34.30 (IO18)
- net LED SDO: now also D1.3 (SDO), D1.4 (SDI), U2.4 (Y); no longer D1.2 (CKO), D1.5 (CKI), U34.31 (IO19)
- net MISO: now also J3.01; no longer J3.03
- net MISO unbuffered: now also U34.19 (IO11); no longer U34.14 (IO12)
- net MOSI: now also J3.03; no longer J3.05
- net MOSI unbuffered: now also U34.22 (IO14); no longer U34.16 (IO13)
- net OE: now also U34.26 (IO45); no longer IC2.8 (OE), U34.28 (IO17)
- net SS10: now also J12.03
- net SS11: now also J12.04
- net SS12: now also J12.06
- net SS13: now also J12.07
- net SS14: now also J12.09
- net SS15: now also J12.10
- net SS16: now also J12.12
- net SS17: now also J2.01
- net SS18: now also J2.03
- net SS19: now also J2.04
- net SS20: now also J2.06
- net SS21: now also J2.07
- net SS22: now also J2.09
- net SS23: now also J2.10
- net SS24: now also J2.12
- net SS9: now also J12.01
- net QRE_OUT: now reaches R2.1, U35.3
- net QRE_OUT: now also U34.15 (IO3); no longer U34.6 (IO34)
- net LED_CLK_unbuffered: now reaches U34.17 (IO9)
- net LED_CLK_unbuffered: now also U1.2 (A)
- net LED_DATA_unbuffered: now reaches U34.18 (IO10)
- net LED_DATA_unbuffered: now also U2.2 (A)
- net at U34.3 (EN): now also C2.1, R3.2, SW2.2
- net UART0_RX: no longer names the net of U34.34 (IO41)
- net UART0_TX: no longer names the net of U34.35 (IO42)
- new net: SW1.2, U34.27 (IO0)
- new net USB_D+: C4.1, J1.2, U34.14 (IO20)
- new net USB_D-: C3.1, J1.3, U34.13 (IO19)
- new net V_BUS: C38.1, IC3.1 (IN), J1.1, JP1.2 (B)
Other:
- note added: "CONNECTORS"
- note added: "LOGIC LEVEL SHIFT FOR APA102"
- note added: "MCU"
- note added: "SPI BUFFER AND MUX"
- moved on the sheet: C34, C35, C36, C37, C38, D1, H1, IC1, IC2, IC3, J10, J11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

Commit message: homework again
Parts:
- C37: footprint Capacitor_SMD:C_0402_1005Metric -> Capacitor_Tantalum_SMD:CP_EIA-3528-15_AVX-H; symbol Device:C -> Device:C_Polarized
- C38: footprint Capacitor_SMD:C_0402_1005Metric -> Capacitor_SMD:C_0603_1608Metric
- J1: footprint digikey-footprints:PinHeader_1x4_P2.54mm_Drill1.02mm -> Connector_PinSocket_2.54mm:PinSocket_1x04_P2.54mm_Horizontal
Connections:
- net GND: now also U34.1 (GND); no longer U34.41 (GND)
- net USB_D+: now also C3.1, J1.3; no longer C4.1, J1.2
- net USB_D-: now also C4.1, J1.2; no longer C3.1, J1.3
- net LED CLK renamed LED_CLK
- net LED SDO renamed LED_DATA
Other:
- moved on the sheet: C3, C4, J1
