File: percussiveInterface-3.2/main_board/main_board_new-3.2.kicad_sch (KiCad schematic)
At the start: 83 parts, among them IC1 ADG731BSUZ, IC2 TXU0304PWR, IC3 LM3940IMP-3.3_NOPB, J1 0022232041, J10 SAMTEC-SLW-108-01-X-S, J11 Screw_Terminal_01x02, J5 SLW-104-01-G-S, J6 SLW-104-01-G-S, J7 SLW-104-01-G-S, J8 SLW-104-01-G-S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

Commit message: jlc board
Parts:
- added H60: MountingHole, MountingHole:MountingHole_3.2mm_M3_DIN965, symbol Mechanical:MountingHole
Connections:
- net OE: no longer names the net of U34.26 (IO45)
Changed lines of the file:
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@@
-    (stroke (width 0) (type default))
-  )
-  (wire (pts (xy 158.75 217.805) (xy 153.67 217.805))
     (stroke (width 0) (type default))
   )
@@
   (label "GND" (at 35.56 196.85 270) (fields_autoplaced)
     (effects (font (size 1.27 1.27)) (justify right bottom))
-  )
-  (label "OE" (at 158.75 217.805 0) (fields_autoplaced)
-    (effects (font (size 1.27 1.27)) (justify left bottom))
   )
   (label "SS22" (at 436.88 298.45 90) (fields_autoplaced)
@@
         )
       )
+    )
+  )
+  (symbol (lib_id "Mechanical:MountingHole") (at 250.825 117.475 0) (unit 1)
+    (in_bom yes) (on_board yes) (dnp no) (fields_autoplaced)
+    (property "Reference" "H60" (at 254 116.205 0)
+      (effects (font (size 1.27 1.27)) (justify left))
+    )
+    (property "Value" "MountingHole" (at 254 118.745 0)
+      (effects (font (size 1.27 1.27)) (justify left))
+    )
+    (property "Footprint" "MountingHole:MountingHole_3.2mm_M3_DIN965" (at 250.825 117.475 0)
+      (effects (font (size 1.27 1.27)) hide)
+    )
+    (property "Datasheet" "~" (at 250.825 117.475 0)
+      (effects (font (size 1.27 1.27)) hide)
+    )
+    (instances
+      (project "main_board_new-3.2"
+        (path "/1e5e0f90-3c6a-4032-b605-c5ae5046b236"
+          (reference "H60") (unit 1)
+        )
+      )
