File: percussiveInterface-3.2/main_board/main_board_new-3.2.kicad_pcb (KiCad board)
At the start: 4 copper layers, 369.4 x 107.4 mm, 199 parts, among them IC1 ADG731BSUZ, IC2 TXU0304PWR, IC3 LM3940IMP-3.3_NOPB, J1 0022232041, J10 SAMTEC-SLW-108-01-X-S, J11 Screw_Terminal_01x02, J5 SLW-104-01-G-S, J6 SLW-104-01-G-S, J7 SLW-104-01-G-S, J8 SLW-104-01-G-S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

Commit message: bremen_workation
Parts:
- moved H12 5.88 mm to (43.6, 222.1)
- moved H13 5.88 mm to (46.1, 222.1)
- moved H14 5.88 mm to (50.6, 222.1)
- moved H15 5.88 mm to (53.1, 222.1)
- moved H16 5.88 mm to (57.6, 222.1)
- moved H17 5.88 mm to (60.1, 222.1)
- moved H18 5.88 mm to (64.6, 222.1)
- moved H19 5.88 mm to (67.1, 222.1)
- moved H20 5.88 mm to (71.6, 222.1)
- moved H21 5.88 mm to (74.1, 222.1)
- moved H22 5.88 mm to (78.6, 222.1)
- moved H23 5.88 mm to (81.1, 222.1)
- moved H24 5.88 mm to (85.6, 222.1)
- moved H25 5.88 mm to (88.1, 222.1)
- moved H26 5.88 mm to (92.6, 222.1)
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Routing:
- net /CLK: track 280.1 -> 286.4 mm
- net /SS2: track 195.1 -> 201.0 mm
- net /SS9: track 104.4 -> 110.2 mm
- net /SS7: track 135.2 -> 141.1 mm
- net /SS5: track 161.5 -> 167.4 mm
- net /SS6: track 145.9 -> 151.8 mm
- net /SS4: track 172.7 -> 178.5 mm
- net /SS3: track 182.2 -> 188.1 mm
- net /SS24: track 16.1 -> 21.9 mm
- net /SS23: track 12.1 -> 18.0 mm
- net /SS22: track 12.6 -> 18.5 mm
- net /SS20: track 23.0 -> 28.8 mm
- net /SS19: track 30.2 -> 36.1 mm
- net /SS17: track 44.7 -> 50.6 mm
- net /SS16: track 51.5 -> 57.3 mm
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