File: percussiveInterface-3.2/magnetometer_array_3/magnetometer_array_3.kicad_pcb (KiCad board)
At the start: 4 copper layers, 8 x 168 mm, 72 parts, among them J1 Conn_01x02_Pin, J10 Conn_01x02_Pin, J11 Conn_01x02_Pin, J12 Conn_01x02_Pin, J13 Conn_01x02_Pin, J14 Conn_01x02_Pin, J15 Conn_01x02_Pin, J16 Conn_01x02_Pin, J17 Conn_01x02_Pin, J18 Conn_01x02_Pin, J19 Conn_01x02_Pin, J2 Conn_01x02_Pin, J20 Conn_01x02_Pin, J21 Conn_01x02_Pin, J22 Conn_01x02_Pin, J23 Conn_01x02_Pin, J24 Conn_01x02_Pin, J3 Conn_01x02_Pin, J4 Conn_01x02_Pin, J5 Conn_01x02_Pin, J6 Conn_01x02_Pin, J7 Conn_01x02_Pin, J8 Conn_01x02_Pin, J9 Conn_01x02_Pin, U1 SM225-10E, U10 SM225-10E, U11 SM225-10E, U12 SM225-10E, U13 SM225-10E, U14 SM225-10E, U15 SM225-10E, U16 SM225-10E, U17 SM225-10E, U18 SM225-10E, U19 SM225-10E, U2 SM225-10E, U20 SM225-10E, U21 SM225-10E, U22 SM225-10E, U23 SM225-10E, U24 SM225-10E, U3 SM225-10E, U4 SM225-10E, U5 SM225-10E, U6 SM225-10E, U7 SM225-10E, U8 SM225-10E, U9 SM225-10E

Commit message: jlc board
Parts:
- moved J24 399.3 mm to (235.2, 90.4), turned to 0 degrees
- moved U24 397.6 mm to (234.3, 89.5), turned to 90 degrees
- moved J23 394.6 mm to (228.2, 90.4), turned to 0 degrees
- moved C24 394.4 mm to (232.0, 88.2), turned to 180 degrees
- moved U23 392.9 mm to (227.3, 89.5), turned to 90 degrees
- moved J22 390.2 mm to (221.2, 90.4), turned to 0 degrees
- moved C23 389.8 mm to (225.0, 88.2), turned to 180 degrees
- moved U22 388.5 mm to (220.3, 89.5), turned to 90 degrees
- moved J21 385.9 mm to (214.2, 90.4), turned to 0 degrees
- moved C22 385.4 mm to (218.0, 88.2), turned to 180 degrees
- moved U21 384.3 mm to (213.3, 89.5), turned to 90 degrees
- moved J20 381.9 mm to (207.2, 90.4), turned to 0 degrees
- moved C21 381.3 mm to (211.0, 88.2), turned to 180 degrees
- moved U20 380.3 mm to (206.3, 89.5), turned to 90 degrees
- moved J19 378.1 mm to (200.2, 90.4), turned to 0 degrees
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Routing:
- net GND: track 37.2 -> 56.0 mm
Other:
- board size 8 x 168 mm -> 168 x 8 mm
