File: percussiveInterface-3.2/new_board_fully_integrated/board_fully_integrated.kicad_pcb (KiCad board)
At the start: 4 copper layers, 369.4 x 107.4 mm, 195 parts, among them IC1 ADG731BSUZ, IC3 LM3940IMP-3.3_NOPB, J1 0022232041, J11 Screw_Terminal_01x02, J6 SLW-104-01-G-S, J8 SLW-104-01-G-S, SW1 SW_Boot, SW2 SW_Reset, U1 SN74LV1T34DBV, U12 TMAG5170, U13 TMAG5170, U14 TMAG5170, U15 TMAG5170, U16 TMAG5170, U17 TMAG5170, U18 TMAG5170, U19 TMAG5170, U2 SN74LV1T34DBV, U20 TMAG5170, U21 TMAG5170, U22 TMAG5170, U23 TMAG5170, U24 TMAG5170, U25 TMAG5170, U26 TMAG5170, U27 TMAG5170, U28 TMAG5170, U29 TMAG5170, U30 TMAG5170, U31 TMAG5170, U32 TMAG5170, U33 TMAG5170, U34 ESP32-S3-WROOM-1-n16r8, U35 QRE1113GR, U36 TMAG5170, U37 TMAG5170, U38 TMAG5170, U39 TMAG5170

Commit message: afaeaefdga
Parts:
- removed D1: APA102-2020, LED_SMD:LED-APA102-2020
- removed the H1 at (329.0, 225.0)
- removed the H1 at (287.0, 225.0)
- removed the H1 at (343.0, 225.0)
- removed the H1 at (385.0, 225.0)
- removed the H1 at (357.0, 225.0)
- removed the H1 at (371.0, 225.0)
- removed the H1 at (301.0, 225.0)
- removed the H1 at (399.0, 225.0)
- removed the H1 at (315.0, 225.0)
- removed J6, J8: SLW-104-01-G-S, Own_Library:SAMTEC_SLW-104-01-G-S
- added C42: 0.1µ, Capacitor_SMD:C_0402_1005Metric, F.Cu at (183.6, 213.2)
- added C43: 0.1µ, Capacitor_SMD:C_0402_1005Metric, F.Cu at (183.6, 215.2)
- added D12: APA102-2020, LED_SMD:LED-APA102-2020, F.Cu at (228.5, 225.0)
- added D13: APA102-2020, LED_SMD:LED-APA102-2020, F.Cu at (375.5, 225.0)
- added D14: APA102-2020, LED_SMD:LED-APA102-2020, F.Cu at (386.0, 225.0)
- added D15: APA102-2020, LED_SMD:LED-APA102-2020, F.Cu at (382.5, 225.0)
- added D16: APA102-2020, LED_SMD:LED-APA102-2020, F.Cu at (379.0, 225.0)
- added D17: APA102-2020, LED_SMD:LED-APA102-2020, F.Cu at (372.0, 225.0)
- added D18: APA102-2020, LED_SMD:LED-APA102-2020, F.Cu at (368.5, 225.0)
- added D19: APA102-2020, LED_SMD:LED-APA102-2020, F.Cu at (365.0, 225.0)
- added D20: APA102-2020, LED_SMD:LED-APA102-2020, F.Cu at (361.5, 225.0)
- added D21: APA102-2020, LED_SMD:LED-APA102-2020, F.Cu at (358.0, 225.0)
- added D22: APA102-2020, LED_SMD:LED-APA102-2020, F.Cu at (354.5, 225.0)
- added D23: APA102-2020, LED_SMD:LED-APA102-2020, F.Cu at (351.0, 225.0)
- added D24: APA102-2020, LED_SMD:LED-APA102-2020, F.Cu at (347.5, 225.0)
- added D25: APA102-2020, LED_SMD:LED-APA102-2020, F.Cu at (344.0, 225.0)
- added D26: APA102-2020, LED_SMD:LED-APA102-2020, F.Cu at (374.6, 219.0)
- added D27: APA102-2020, LED_SMD:LED-APA102-2020, F.Cu at (377.5, 219.0)
- added D28: APA102-2020, LED_SMD:LED-APA102-2020, F.Cu at (380.3, 219.0)
- added D29: APA102-2020, LED_SMD:LED-APA102-2020, F.Cu at (383.2, 219.0)
- added D30: APA102-2020, LED_SMD:LED-APA102-2020, F.Cu at (386.0, 219.0)
- added D31: APA102-2020, LED_SMD:LED-APA102-2020, F.Cu at (388.9, 219.0)
- added D32: APA102-2020, LED_SMD:LED-APA102-2020, F.Cu at (391.8, 219.0)
- added D33: APA102-2020, LED_SMD:LED-APA102-2020, F.Cu at (394.6, 219.0)
- added D34: APA102-2020, LED_SMD:LED-APA102-2020, F.Cu at (397.5, 219.0)
- added D35: APA102-2020, LED_SMD:LED-APA102-2020, F.Cu at (400.3, 219.0)
- added D36: APA102-2020, LED_SMD:LED-APA102-2020, F.Cu at (403.2, 219.0)
- added D37: APA102-2020, LED_SMD:LED-APA102-2020, F.Cu at (406.1, 219.0)
- added D38: APA102-2020, LED_SMD:LED-APA102-2020, F.Cu at (408.9, 219.0)
- added D39: APA102-2020, LED_SMD:LED-APA102-2020, F.Cu at (411.8, 219.0)
- added D40: APA102-2020, LED_SMD:LED-APA102-2020, F.Cu at (414.7, 219.0)
- added D41: APA102-2020, LED_SMD:LED-APA102-2020, F.Cu at (337.0, 225.0)
- added D42: APA102-2020, LED_SMD:LED-APA102-2020, F.Cu at (417.5, 219.9)
- added D43: APA102-2020, LED_SMD:LED-APA102-2020, F.Cu at (272.0, 210.5)
- added D44: APA102-2020, LED_SMD:LED-APA102-2020, F.Cu at (232.0, 225.0)
- added D45: APA102-2020, LED_SMD:LED-APA102-2020, F.Cu at (239.0, 225.0)
- added D46: APA102-2020, LED_SMD:LED-APA102-2020, F.Cu at (284.5, 225.0)
- added D47: APA102-2020, LED_SMD:LED-APA102-2020, F.Cu at (340.5, 225.0)
- added D48: APA102-2020, LED_SMD:LED-APA102-2020, F.Cu at (242.7, 225.0)
- added D49: APA102-2020, LED_SMD:LED-APA102-2020, F.Cu at (246.0, 225.0)
- added D50: APA102-2020, LED_SMD:LED-APA102-2020, F.Cu at (249.5, 225.0)
- added D51: APA102-2020, LED_SMD:LED-APA102-2020, F.Cu at (253.0, 225.0)
- added D52: APA102-2020, LED_SMD:LED-APA102-2020, F.Cu at (256.5, 225.0)
- added D53: APA102-2020, LED_SMD:LED-APA102-2020, F.Cu at (260.0, 225.0)
- added D54: APA102-2020, LED_SMD:LED-APA102-2020, F.Cu at (263.5, 225.0)
- added D55: APA102-2020, LED_SMD:LED-APA102-2020, F.Cu at (267.0, 225.0)
- added D56: APA102-2020, LED_SMD:LED-APA102-2020, F.Cu at (270.5, 225.0)
- added D57: APA102-2020, LED_SMD:LED-APA102-2020, F.Cu at (274.0, 225.0)
- added D58: APA102-2020, LED_SMD:LED-APA102-2020, F.Cu at (277.5, 225.0)
- added D59: APA102-2020, LED_SMD:LED-APA102-2020, F.Cu at (235.5, 225.0)
- added D60: APA102-2020, LED_SMD:LED-APA102-2020, F.Cu at (288.0, 225.0)
- added D61: APA102-2020, LED_SMD:LED-APA102-2020, F.Cu at (281.1, 225.0)
- added D62: APA102-2020, LED_SMD:LED-APA102-2020, F.Cu at (291.5, 225.0)
- added D63: APA102-2020, LED_SMD:LED-APA102-2020, F.Cu at (295.0, 225.0)
- added D64: APA102-2020, LED_SMD:LED-APA102-2020, F.Cu at (298.5, 225.0)
- added D65: APA102-2020, LED_SMD:LED-APA102-2020, F.Cu at (302.0, 225.0)
- added D66: APA102-2020, LED_SMD:LED-APA102-2020, F.Cu at (305.5, 225.0)
- added D67: APA102-2020, LED_SMD:LED-APA102-2020, F.Cu at (309.0, 225.0)
- added D68: APA102-2020, LED_SMD:LED-APA102-2020, F.Cu at (312.5, 225.0)
- added D69: APA102-2020, LED_SMD:LED-APA102-2020, F.Cu at (316.0, 225.0)
- added D70: APA102-2020, LED_SMD:LED-APA102-2020, F.Cu at (319.5, 225.0)
- added D71: APA102-2020, LED_SMD:LED-APA102-2020, F.Cu at (323.0, 225.0)
- added D72: APA102-2020, LED_SMD:LED-APA102-2020, F.Cu at (326.5, 225.0)
- added D73: APA102-2020, LED_SMD:LED-APA102-2020, F.Cu at (330.0, 225.0)
- added D74: APA102-2020, LED_SMD:LED-APA102-2020, F.Cu at (333.5, 225.0)
- added IC2: TXU0304PWR, Own_Library:QFN_04RUTR_TEX, F.Cu at (217.0, 234.0)
- added R12: 10K, Resistor_SMD:R_0402_1005Metric, F.Cu at (223.7, 220.8)
- added R13: 100, Resistor_SMD:R_0402_1005Metric, F.Cu at (224.9, 220.7)
- added U40: QRE1113GR, OptoDevice:OnSemi_CASE100CY, F.Cu at (225.0, 225.0)
- locked: renamed from U1; value SN74LV1T34DBV -> locked
- locked: renamed from U2; value SN74LV1T34DBV -> locked
- moved C35 4.33 mm to (216.5, 236.3), turned to 180 degrees
- moved locked 2.97 mm to (230.5, 230.8)
- moved C6 2.97 mm to (227.7, 231.1)
- moved locked 2.97 mm to (236.3, 230.8)
- moved C5 2.97 mm to (233.4, 231.1)
- moved C13 1.00 mm to (43.5, 220.0)
- moved C14 1.00 mm to (50.5, 220.0)
- moved U12 1.00 mm to (43.0, 225.0)
- moved U13 1.00 mm to (57.0, 225.0)
- moved U14 1.00 mm to (71.0, 225.0)
- moved U15 1.00 mm to (85.0, 225.0)
- moved U16 1.00 mm to (50.0, 225.0)
- moved U17 1.00 mm to (64.0, 225.0)
- moved U18 1.00 mm to (78.0, 225.0)
- moved U19 1.00 mm to (92.0, 225.0)
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Connections:
- IC1 pad 33: /SS25 -> /SS29
- IC1 pad 34: /SS26 -> /SS30
- IC1 pad 35: /SS27 -> /SS31
- IC1 pad 36: /SS28 -> /SS32
- IC1 pad 37: /SS29 -> /SS28
- IC1 pad 38: /SS30 -> /SS27
- IC1 pad 39: /SS31 -> /SS26
- IC1 pad 40: /SS32 -> /SS25
- U34 pad 15: /QRE_OUT -> unconnected-(U34-IO3-Pad15)
- U34 pad 19: /MISO unbuffered -> unconnected-(U34-IO11-Pad19)
- U34 pad 20: /CS1 unbuffered -> /QRE_VIBRO_OUT
- U34 pad 21: /CLK unbuffered -> unconnected-(U34-IO13-Pad21)
- U34 pad 22: /MOSI unbuffered -> /MISO unbuffered
- U34 pad 23: unconnected-(U34-IO21-Pad23) -> /CS1 unbuffered
- U34 pad 24: unconnected-(U34-IO47-Pad24) -> /CLK unbuffered
- U34 pad 25: unconnected-(U34-IO48-Pad25) -> /MOSI unbuffered
- U34 pad 6: unconnected-(U34-IO6-Pad6) -> /QRE_OUT
- U34 pad 8: /LDC_CS -> unconnected-(U34-IO15-Pad8)
- U34 pad 9: /LDC_INT -> unconnected-(U34-IO16-Pad9)
- U38 pad 4: unconnected-(U38-~{CS}-Pad4) -> /SS25
- U39 pad 4: unconnected-(U39-~{CS}-Pad4) -> /SS26
Routing:
- net /SS26: track 0.00 -> 31.9 mm, vias 0 -> 2
- net /SS25: track 0.00 -> 24.4 mm, vias 0 -> 2
- net /CS1: track 4.95 -> 25.5 mm
- net /QRE_VIBRO_OUT: track 0.00 -> 18.4 mm
- net /CLK: track 248.7 -> 256.9 mm
- net /MOSI: track 253.2 -> 260.0 mm
- net Net-(U40-A): track 0.00 -> 6.16 mm
- net /V_BUS: track 36.8 -> 32.2 mm, vias 0 -> 1
- net /LED_CLK_unbuffered: track 9.05 -> 12.4 mm
- net /MISO: track 280.5 -> 277.4 mm
- net /3.3V: track 73.9 -> 71.2 mm
- net /LED_DATA_unbuffered: track 7.15 -> 8.48 mm
- net Net-(U35-A): track 9.86 -> 8.63 mm
- net /SS24: track 20.3 -> 19.1 mm
- net unconnected-(U39-~{CS}-Pad4): track 1.17 -> 0.00 mm, vias 1 -> 0
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