File: percussiveInterface-3.2/new_board_fully_integrated/board_fully_integrated.kicad_sch (KiCad schematic)
At the start: 100 parts, among them IC1 ADG731BSUZ, IC2 TXU0304PWR, IC3 LM3940IMP-3.3_NOPB, J1 0022232041, J10 SAMTEC-SLW-108-01-X-S, J11 Screw_Terminal_01x02, J5 SLW-104-01-G-S, J6 SLW-104-01-G-S, J7 SLW-104-01-G-S, J8 SLW-104-01-G-S, J9 SAMTEC-SLW-108-01-X-S, SW1 SW_Boot, SW2 SW_Reset, U1 SN74LV1T34DBV, U12 TMAG5170, U13 TMAG5170, U14 TMAG5170, U15 TMAG5170, U16 TMAG5170, U17 TMAG5170, U18 TMAG5170, U19 TMAG5170, U2 SN74LV1T34DBV, U20 TMAG5170, U21 TMAG5170, U22 TMAG5170, U23 TMAG5170, U24 TMAG5170, U25 TMAG5170, U26 TMAG5170, U27 TMAG5170, U28 TMAG5170, U29 TMAG5170, U30 TMAG5170, U31 TMAG5170, U32 TMAG5170, U33 TMAG5170, U34 ESP32-S3-WROOM-1-n16r8, U35 QRE1113GR, U36 TMAG5170, U37 TMAG5170, U38 TMAG5170, U39 TMAG5170, U40 TMAG5170, U41 TMAG5170, U42 TMAG5170, U43 TMAG5170, U44 TMAG5170, U45 TMAG5170

Commit message: afaeaefdga
Parts:
- removed C12, C44, C45, C46, C47, C48, C49: 0.1µ, Capacitor_SMD:C_0402_1005Metric, symbol Device:C_Small
- removed D1: APA102-2020, LED_SMD:LED-APA102-2020, symbol LED:APA102-2020
- removed J10, J9: SAMTEC-SLW-108-01-X-S, Own_Library:SAMTEC-SLW-108-01-X-S, symbol SAMTEC-SLW-108-01-X-S:SAMTEC-SLW-108-01-X-S
- removed J5, J6, J7, J8: SLW-104-01-G-S, Own_Library:SAMTEC_SLW-104-01-G-S, symbol SLW-104-01-G-S:SLW-104-01-G-S
- removed U40, U41, U42, U43, U44, U45: TMAG5170, Package_SO:VSSOP-8_3.0x3.0mm_P0.65mm, symbol Sensor_Magnetic:TMAG5170-Q1
- added D12, D13, D14, D15, D16, D17, D18, D19, D20, D21, D22, D23, D24, D25, D26, D27, D28, D29, D30, D31, D32, D33, D34, D35, D36, D37, D38, D39, D40, D41, D42, D43, D44, D45, D46, D47, D48, D49, D50, D51, D52, D53, D54, D55, D56, D57, D58, D59, D60, D61, D62, D63, D64, D65, D66, D67, D68, D69, D70, D71, D72, D73, D74: APA102-2020, LED_SMD:LED-APA102-2020, symbol LED:APA102-2020
- added R12: 10K, Resistor_SMD:R_0402_1005Metric, symbol Device:R
- added R13: 100, Resistor_SMD:R_0402_1005Metric, symbol Device:R
- added U40: QRE1113GR, OptoDevice:OnSemi_CASE100CY, symbol Sensor_Proximity:QRE1113GR
- IC2: footprint Package_SO:TSSOP-14_4.4x5mm_P0.65mm -> QFN_04RUTR_TEX; symbol TXU0304PWR:TXU0304PWR -> TXU0304RUTR:TXU0304RUTR
Connections:
- net 3.3V: now also IC2.11 (VCCB), IC2.12 (OE), R12.2, R13.1; no longer IC2.14 (VCCB), IC2.8 (OE)
- net 5V: now also D12.1 (VDD), D13.1 (VDD), D14.1 (VDD), D15.1 (VDD), D16.1 (VDD), D17.1 (VDD), D18.1 (VDD), D19.1 (VDD), D20.1 (VDD), D21.1 (VDD), D22.1 (VDD), D23.1 (VDD), D24.1 (VDD), D25.1 (VDD), D26.1 (VDD), D27.1 (VDD), D28.1 (VDD), D29.1 (VDD), D30.1 (VDD), D31.1 (VDD), D32.1 (VDD), D33.1 (VDD), D34.1 (VDD), D35.1 (VDD), D36.1 (VDD), D37.1 (VDD), D38.1 (VDD), D39.1 (VDD), D40.1 (VDD), D41.1 (VDD), D42.1 (VDD), D43.1 (VDD), D44.1 (VDD), D45.1 (VDD), D46.1 (VDD), D47.1 (VDD), D48.1 (VDD), D49.1 (VDD), D50.1 (VDD), D51.1 (VDD), D52.1 (VDD), D53.1 (VDD), D54.1 (VDD), D55.1 (VDD), D56.1 (VDD), D57.1 (VDD), D58.1 (VDD), D59.1 (VDD), D60.1 (VDD), D61.1 (VDD), D62.1 (VDD), D63.1 (VDD), D64.1 (VDD), D65.1 (VDD), D66.1 (VDD), D67.1 (VDD), D68.1 (VDD), D69.1 (VDD), D70.1 (VDD), D71.1 (VDD), D72.1 (VDD), D73.1 (VDD), D74.1 (VDD)
- net CLK: now also IC2.9 (B2Y); no longer IC2.12 (B2Y)
- net CLK unbuffered: now also U34.24 (IO47); no longer U34.21 (IO13)
- net CS1: now also IC2.8 (B3Y); no longer IC2.11 (B3Y)
- net CS1 unbuffered: now also U34.23 (IO21); no longer U34.20 (IO12)
- net GND: now also IC2.6 (GND), D12.6 (GND), D13.6 (GND), D14.6 (GND), D15.6 (GND), D16.6 (GND), D17.6 (GND), D18.6 (GND), D19.6 (GND), D20.6 (GND), D21.6 (GND), D22.6 (GND), D23.6 (GND), D24.6 (GND), D25.6 (GND), D26.6 (GND), D27.6 (GND), D28.6 (GND), D29.6 (GND), D30.6 (GND), D31.6 (GND), D32.6 (GND), D33.6 (GND), D34.6 (GND), D35.6 (GND), D36.6 (GND), D37.6 (GND), D38.6 (GND), D39.6 (GND), D40.6 (GND), D41.6 (GND), D42.6 (GND), D43.6 (GND), D44.6 (GND), D45.6 (GND), D46.6 (GND), D47.6 (GND), D48.6 (GND), D49.6 (GND), D50.6 (GND), D51.6 (GND), D52.6 (GND), D53.6 (GND), D54.6 (GND), D55.6 (GND), D56.6 (GND), D57.6 (GND), D58.6 (GND), D59.6 (GND), D60.6 (GND), D61.6 (GND), D62.6 (GND), D63.6 (GND), D64.6 (GND), D65.6 (GND), D66.6 (GND), D67.6 (GND), D68.6 (GND), D69.6 (GND), D70.6 (GND), D71.6 (GND), D72.6 (GND), D73.6 (GND), D74.6 (GND), U40.2 (K), U40.4; no longer IC2.7 (GND)
- net LED_CLK: now also D12.2 (CKO), D12.5 (CKI), D13.2 (CKO), D13.5 (CKI), D14.2 (CKO), D14.5 (CKI), D15.2 (CKO), D15.5 (CKI), D16.2 (CKO), D16.5 (CKI), D17.2 (CKO), D17.5 (CKI), D18.2 (CKO), D18.5 (CKI), D19.2 (CKO), D19.5 (CKI), D20.2 (CKO), D20.5 (CKI), D21.2 (CKO), D21.5 (CKI), D22.2 (CKO), D22.5 (CKI), D23.2 (CKO), D23.5 (CKI), D24.2 (CKO), D24.5 (CKI), D25.2 (CKO), D25.5 (CKI), D26.2 (CKO), D26.5 (CKI), D27.2 (CKO), D27.5 (CKI), D28.2 (CKO), D28.5 (CKI), D29.2 (CKO), D29.5 (CKI), D30.2 (CKO), D30.5 (CKI), D31.2 (CKO), D31.5 (CKI), D32.2 (CKO), D32.5 (CKI), D33.2 (CKO), D33.5 (CKI), D34.2 (CKO), D34.5 (CKI), D35.2 (CKO), D35.5 (CKI), D36.2 (CKO), D36.5 (CKI), D37.2 (CKO), D37.5 (CKI), D38.2 (CKO), D38.5 (CKI), D39.2 (CKO), D39.5 (CKI), D40.2 (CKO), D40.5 (CKI), D41.2 (CKO), D41.5 (CKI), D42.2 (CKO), D42.5 (CKI), D43.2 (CKO), D43.5 (CKI), D44.2 (CKO), D44.5 (CKI), D45.2 (CKO), D45.5 (CKI), D46.2 (CKO), D46.5 (CKI), D47.2 (CKO), D47.5 (CKI), D48.2 (CKO), D48.5 (CKI), D49.2 (CKO), D49.5 (CKI), D50.2 (CKO), D50.5 (CKI), D51.2 (CKO), D51.5 (CKI), D52.2 (CKO), D52.5 (CKI), D53.2 (CKO), D53.5 (CKI), D54.2 (CKO), D54.5 (CKI), D55.2 (CKO), D55.5 (CKI), D56.2 (CKO), D56.5 (CKI), D57.2 (CKO), D57.5 (CKI), D58.2 (CKO), D58.5 (CKI), D59.2 (CKO), D59.5 (CKI), D60.2 (CKO), D60.5 (CKI), D61.2 (CKO), D61.5 (CKI), D62.2 (CKO), D62.5 (CKI), D63.2 (CKO), D63.5 (CKI), D64.2 (CKO), D64.5 (CKI), D65.2 (CKO), D65.5 (CKI), D66.2 (CKO), D66.5 (CKI), D67.2 (CKO), D67.5 (CKI), D68.2 (CKO), D68.5 (CKI), D69.2 (CKO), D69.5 (CKI), D70.2 (CKO), D70.5 (CKI), D71.2 (CKO), D71.5 (CKI), D72.2 (CKO), D72.5 (CKI), D73.2 (CKO), D73.5 (CKI), D74.2 (CKO), D74.5 (CKI)
- net LED_DATA: now also D12.3 (SDO), D12.4 (SDI), D13.3 (SDO), D13.4 (SDI), D14.3 (SDO), D14.4 (SDI), D15.3 (SDO), D15.4 (SDI), D16.3 (SDO), D16.4 (SDI), D17.3 (SDO), D17.4 (SDI), D18.3 (SDO), D18.4 (SDI), D19.3 (SDO), D19.4 (SDI), D20.3 (SDO), D20.4 (SDI), D21.3 (SDO), D21.4 (SDI), D22.3 (SDO), D22.4 (SDI), D23.3 (SDO), D23.4 (SDI), D24.3 (SDO), D24.4 (SDI), D25.3 (SDO), D25.4 (SDI), D26.3 (SDO), D26.4 (SDI), D27.3 (SDO), D27.4 (SDI), D28.3 (SDO), D28.4 (SDI), D29.3 (SDO), D29.4 (SDI), D30.3 (SDO), D30.4 (SDI), D31.3 (SDO), D31.4 (SDI), D32.3 (SDO), D32.4 (SDI), D33.3 (SDO), D33.4 (SDI), D34.3 (SDO), D34.4 (SDI), D35.3 (SDO), D35.4 (SDI), D36.3 (SDO), D36.4 (SDI), D37.3 (SDO), D37.4 (SDI), D38.3 (SDO), D38.4 (SDI), D39.3 (SDO), D39.4 (SDI), D40.3 (SDO), D40.4 (SDI), D41.3 (SDO), D41.4 (SDI), D42.3 (SDO), D42.4 (SDI), D43.3 (SDO), D43.4 (SDI), D44.3 (SDO), D44.4 (SDI), D45.3 (SDO), D45.4 (SDI), D46.3 (SDO), D46.4 (SDI), D47.3 (SDO), D47.4 (SDI), D48.3 (SDO), D48.4 (SDI), D49.3 (SDO), D49.4 (SDI), D50.3 (SDO), D50.4 (SDI), D51.3 (SDO), D51.4 (SDI), D52.3 (SDO), D52.4 (SDI), D53.3 (SDO), D53.4 (SDI), D54.3 (SDO), D54.4 (SDI), D55.3 (SDO), D55.4 (SDI), D56.3 (SDO), D56.4 (SDI), D57.3 (SDO), D57.4 (SDI), D58.3 (SDO), D58.4 (SDI), D59.3 (SDO), D59.4 (SDI), D60.3 (SDO), D60.4 (SDI), D61.3 (SDO), D61.4 (SDI), D62.3 (SDO), D62.4 (SDI), D63.3 (SDO), D63.4 (SDI), D64.3 (SDO), D64.4 (SDI), D65.3 (SDO), D65.4 (SDI), D66.3 (SDO), D66.4 (SDI), D67.3 (SDO), D67.4 (SDI), D68.3 (SDO), D68.4 (SDI), D69.3 (SDO), D69.4 (SDI), D70.3 (SDO), D70.4 (SDI), D71.3 (SDO), D71.4 (SDI), D72.3 (SDO), D72.4 (SDI), D73.3 (SDO), D73.4 (SDI), D74.3 (SDO), D74.4 (SDI)
- net MISO: now also IC2.7 (B4); no longer IC2.10 (B4)
- net MISO unbuffered: now also U34.22 (IO14); no longer U34.19 (IO11)
- net MOSI: now also IC2.10 (B1Y); no longer IC2.13 (B1Y)
- net MOSI unbuffered: now also U34.25 (IO48); no longer U34.22 (IO14)
- net QRE_OUT: now also U34.6 (IO6); no longer U34.15 (IO3)
- net SS25: now also IC1.40 (S32), U38.4 (~{CS}); no longer IC1.33 (S25)
- net SS26: now also IC1.39 (S31), U39.4 (~{CS}); no longer IC1.34 (S26)
- net SS27: now also IC1.38 (S30); no longer IC1.35 (S27)
- net SS28: now also IC1.37 (S29); no longer IC1.36 (S28)
- net SS29: now also IC1.33 (S25); no longer IC1.37 (S29)
- net SS30: now also IC1.34 (S26); no longer IC1.38 (S30)
- net SS31: now also IC1.35 (S27); no longer IC1.39 (S31)
- net SS32: now also IC1.36 (S28); no longer IC1.40 (S32)
- net LDC_CS: no longer names the net of U34.8 (IO15)
- net LDC_INT: no longer names the net of U34.9 (IO16)
- new net: R13.2, U40.1 (A)
- new net QRE_VIBRO_OUT: R12.1, U34.20 (IO12), U40.3
Other:
- note added: "LEDS"
- note added: "REFLECTIVE VIBROMETER"
- note removed: "CONNECTORS"
- moved on the sheet: C1, C13, C14, C15, C16, C17, C18, C19, C2, C20, C21, C22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

Commit message: asgfebgsdfbas
Parts:
- removed D25, D26, D27, D28, D29, D30, D31, D32, D33, D34, D35, D36, D37, D38, D39, D40, D41, D70, D71, D72, D73, D74: APA102-2020, LED_SMD:LED-APA102-2020, symbol LED:APA102-2020
- added C36, C37, C38, C39, C40, C41, C42, C43, C44, C45, C46, C47, C48, C49, C50, C51, C52, C53, C54, C55, C56, C57, C58, C59, C60, C61, C64, C65: 0.1µ, Capacitor_SMD:C_0402_1005Metric, symbol Device:C_Small
- added C66: 680µF, Capacitor_Tantalum_SMD:CP_EIA-7343-30_AVX-N, symbol Device:C_Polarized
- added D44, D45, D46, D47, D48, D49, D50, D51, D52, D53, D54: APA102-2020, Own_Library:LED-APA102-2020, symbol LED:APA102-2020
- added H4, H5, H6: MountingHole, MountingHole:MountingHole_3.2mm_M3_DIN965, symbol Mechanical:MountingHole
- added IC4: ADG731BSUZ, Package_QFP:TQFP-48_7x7mm_P0.5mm, symbol ADG731BSUZ:ADG731BSUZ
- added IC5: TXU0304PWR, Own_Library:QFN_04RUTR_TEX, symbol TXU0304RUTR:TXU0304RUTR
- added U30, U31, U32, U33, U34, U36, U37, U38, U39, U41, U42, U43, U44, U45, U46, U47, U48, U49, U50, U51, U52, U53, U54, U55, U56, U57: TMAG5170, Package_SO:VSSOP-8_3.0x3.0mm_P0.65mm, symbol Sensor_Magnetic:TMAG5170-Q1
- D10: renamed from D19; footprint LED_SMD:LED-APA102-2020 -> Own_Library:LED-APA102-2020
- D11: renamed from D20; footprint LED_SMD:LED-APA102-2020 -> Own_Library:LED-APA102-2020
- D12: renamed from D21; footprint LED_SMD:LED-APA102-2020 -> Own_Library:LED-APA102-2020
- D13: renamed from D22; footprint LED_SMD:LED-APA102-2020 -> Own_Library:LED-APA102-2020
- D14: renamed from D23; footprint LED_SMD:LED-APA102-2020 -> Own_Library:LED-APA102-2020
- D15: renamed from D24; footprint LED_SMD:LED-APA102-2020 -> Own_Library:LED-APA102-2020
- D16: renamed from D44; footprint LED_SMD:LED-APA102-2020 -> Own_Library:LED-APA102-2020
- D17: renamed from D46; footprint LED_SMD:LED-APA102-2020 -> Own_Library:LED-APA102-2020
- D18: renamed from D48; footprint LED_SMD:LED-APA102-2020 -> Own_Library:LED-APA102-2020
- D19: renamed from D50; footprint LED_SMD:LED-APA102-2020 -> Own_Library:LED-APA102-2020
- D20: renamed from D52; footprint LED_SMD:LED-APA102-2020 -> Own_Library:LED-APA102-2020
- D21: renamed from D54; footprint LED_SMD:LED-APA102-2020 -> Own_Library:LED-APA102-2020
- D22: renamed from D56; footprint LED_SMD:LED-APA102-2020 -> Own_Library:LED-APA102-2020
- D23: renamed from D58; footprint LED_SMD:LED-APA102-2020 -> Own_Library:LED-APA102-2020
- D24: renamed from D60; footprint LED_SMD:LED-APA102-2020 -> Own_Library:LED-APA102-2020
- D25: renamed from D62; footprint LED_SMD:LED-APA102-2020 -> Own_Library:LED-APA102-2020
- D26: renamed from D64; footprint LED_SMD:LED-APA102-2020 -> Own_Library:LED-APA102-2020
- D27: renamed from D66; footprint LED_SMD:LED-APA102-2020 -> Own_Library:LED-APA102-2020
- D28: renamed from D68; footprint LED_SMD:LED-APA102-2020 -> Own_Library:LED-APA102-2020
- D29: renamed from D45; footprint LED_SMD:LED-APA102-2020 -> Own_Library:LED-APA102-2020
- D3: renamed from D12; footprint LED_SMD:LED-APA102-2020 -> Own_Library:LED-APA102-2020
- D30: renamed from D47; footprint LED_SMD:LED-APA102-2020 -> Own_Library:LED-APA102-2020
- D31: renamed from D49; footprint LED_SMD:LED-APA102-2020 -> Own_Library:LED-APA102-2020
- D32: renamed from D51; footprint LED_SMD:LED-APA102-2020 -> Own_Library:LED-APA102-2020
- D33: renamed from D53; footprint LED_SMD:LED-APA102-2020 -> Own_Library:LED-APA102-2020
- D34: renamed from D55; footprint LED_SMD:LED-APA102-2020 -> Own_Library:LED-APA102-2020
- D35: renamed from D57; footprint LED_SMD:LED-APA102-2020 -> Own_Library:LED-APA102-2020
- D36: renamed from D59; footprint LED_SMD:LED-APA102-2020 -> Own_Library:LED-APA102-2020
- D37: renamed from D61; footprint LED_SMD:LED-APA102-2020 -> Own_Library:LED-APA102-2020
- D38: renamed from D63; footprint LED_SMD:LED-APA102-2020 -> Own_Library:LED-APA102-2020
- D39: renamed from D65; footprint LED_SMD:LED-APA102-2020 -> Own_Library:LED-APA102-2020
- D4: renamed from D13; footprint LED_SMD:LED-APA102-2020 -> Own_Library:LED-APA102-2020
- D40: renamed from D67; footprint LED_SMD:LED-APA102-2020 -> Own_Library:LED-APA102-2020
- D41: renamed from D69; footprint LED_SMD:LED-APA102-2020 -> Own_Library:LED-APA102-2020
- D42, D43: footprint LED_SMD:LED-APA102-2020 -> Own_Library:LED-APA102-2020
- D5: renamed from D14; footprint LED_SMD:LED-APA102-2020 -> Own_Library:LED-APA102-2020
- D6: renamed from D15; footprint LED_SMD:LED-APA102-2020 -> Own_Library:LED-APA102-2020
- D7: renamed from D16; footprint LED_SMD:LED-APA102-2020 -> Own_Library:LED-APA102-2020
- D8: renamed from D17; footprint LED_SMD:LED-APA102-2020 -> Own_Library:LED-APA102-2020
- D9: renamed from D18; footprint LED_SMD:LED-APA102-2020 -> Own_Library:LED-APA102-2020
- H1: value MountingHole_Pad -> MountingHole
- IC2: footprint QFN_04RUTR_TEX -> Own_Library:QFN_04RUTR_TEX
- renumbered C38 to C1, C13 to C10, C14 to C11, C15 to C12, C16 to C13, C21 to C14, C23 to C15, C25 to C16, C27 to C17, C29 to C18, C31 to C19, C34 to C2, C33 to C20, C40 to C21, C42 to C22, C17 to C23, C18 to C24, C19 to C25, C20 to C26, C22 to C27, C24 to C28, C26 to C29, C1 to C3, C28 to C30, C30 to C31, C39 to C33, C41 to C34, C43 to C35, C36 to C4, C37 to C5, C35 to C6, C4 to C62, C6 to C63, C2 to C7, C3 to C8, C5 to C9, H60 to H3, U15 to U10, U19 to U11, U20 to U12, U21 to U13, U22 to U14, U23 to U15, U24 to U16, U25 to U17, U26 to U18, U27 to U19, U28 to U20, U29 to U21, U30 to U22, U31 to U23, U32 to U24, U33 to U25, U36 to U26, U37 to U27, U38 to U28, U39 to U29, U12 to U4, U16 to U5, U13 to U6, U34 to U60, U40 to U61, U17 to U7, U14 to U8, U18 to U9
Connections:
- net 3.3V: now also C36.2, C37.2, C38.2, C39.2, C40.2, C41.2, C42.2, C43.2, C44.2, C45.2, C46.2, C47.2, C48.2, C49.2, C50.2, C51.2, C52.2, C53.2, C54.2, C55.2, C56.2, C57.2, C58.2, C59.2, C60.2, C61.2, C64.1, C65.1, IC4.13 (VDD_1), IC4.14 (VDD_2), IC5.1 (VCCA), IC5.11 (VCCB), IC5.12 (OE), U30.5 (VCC), U31.5 (VCC), U32.5 (VCC), U33.5 (VCC), U34.5 (VCC), U36.5 (VCC), U37.5 (VCC), U38.5 (VCC), U39.5 (VCC), U41.5 (VCC), U42.5 (VCC), U43.5 (VCC), U44.5 (VCC), U45.5 (VCC), U46.5 (VCC), U47.5 (VCC), U48.5 (VCC), U49.5 (VCC), U50.5 (VCC), U51.5 (VCC), U52.5 (VCC), U53.5 (VCC), U54.5 (VCC), U55.5 (VCC), U56.5 (VCC), U57.5 (VCC)
- net 5V: now also C66.1, D44.1 (VDD), D45.1 (VDD), D46.1 (VDD), D47.1 (VDD), D48.1 (VDD), D49.1 (VDD), D50.1 (VDD), D51.1 (VDD), D52.1 (VDD), D53.1 (VDD), D54.1 (VDD)
- net CLK: now also IC4.19 (SCLK), IC5.9 (B2Y), U30.1 (SCLK), U31.1 (SCLK), U32.1 (SCLK), U33.1 (SCLK), U34.1 (SCLK), U36.1 (SCLK), U37.1 (SCLK), U38.1 (SCLK), U39.1 (SCLK), U41.1 (SCLK), U42.1 (SCLK), U43.1 (SCLK), U44.1 (SCLK), U45.1 (SCLK), U46.1 (SCLK), U47.1 (SCLK), U48.1 (SCLK), U49.1 (SCLK), U50.1 (SCLK), U51.1 (SCLK), U52.1 (SCLK), U53.1 (SCLK), U54.1 (SCLK), U55.1 (SCLK), U56.1 (SCLK), U57.1 (SCLK)
- net CLK unbuffered: now also IC5.3 (A2)
- net CS1: now also IC4.43 (D), IC5.8 (B3Y)
- net CS1 unbuffered: now also IC5.4 (A3)
- net GND: now also C36.1, C37.1, C38.1, C39.1, C40.1, C41.1, C42.1, C43.1, C44.1, C45.1, C46.1, C47.1, C48.1, C49.1, C50.1, C51.1, C52.1, C53.1, C54.1, C55.1, C56.1, C57.1, C58.1, C59.1, C60.1, C61.1, C64.2, C65.2, C66.2, D44.6 (GND), D45.6 (GND), D46.6 (GND), D47.6 (GND), D48.6 (GND), D49.6 (GND), D50.6 (GND), D51.6 (GND), D52.6 (GND), D53.6 (GND), D54.6 (GND), IC4.23 (GND), IC4.24 (VSS), IC5.6 (GND), U30.6 (GND), U30.7 (TEST), U31.6 (GND), U31.7 (TEST), U32.6 (GND), U32.7 (TEST), U33.6 (GND), U33.7 (TEST), U34.6 (GND), U34.7 (TEST), U36.6 (GND), U36.7 (TEST), U37.6 (GND), U37.7 (TEST), U38.6 (GND), U38.7 (TEST), U39.6 (GND), U39.7 (TEST), U41.6 (GND), U41.7 (TEST), U42.6 (GND), U42.7 (TEST), U43.6 (GND), U43.7 (TEST), U44.6 (GND), U44.7 (TEST), U45.6 (GND), U45.7 (TEST), U46.6 (GND), U46.7 (TEST), U47.6 (GND), U47.7 (TEST), U48.6 (GND), U48.7 (TEST), U49.6 (GND), U49.7 (TEST), U50.6 (GND), U50.7 (TEST), U51.6 (GND), U51.7 (TEST), U52.6 (GND), U52.7 (TEST), U53.6 (GND), U53.7 (TEST), U54.6 (GND), U54.7 (TEST), U55.6 (GND), U55.7 (TEST), U56.6 (GND), U56.7 (TEST), U57.6 (GND), U57.7 (TEST)
- net LED_CLK: now also D44.2 (CKO), D44.5 (CKI), D45.2 (CKO), D45.5 (CKI), D46.2 (CKO), D46.5 (CKI), D47.2 (CKO), D47.5 (CKI), D48.2 (CKO), D48.5 (CKI), D49.2 (CKO), D49.5 (CKI), D50.2 (CKO), D50.5 (CKI), D51.2 (CKO), D51.5 (CKI), D52.2 (CKO), D52.5 (CKI), D53.2 (CKO), D53.5 (CKI), D54.2 (CKO), D54.5 (CKI)
- net LED_CLK_unbuffered: now also U60.20 (IO12); no longer U60.17 (IO9)
- net LED_DATA: now also D44.3 (SDO), D44.4 (SDI), D45.3 (SDO), D45.4 (SDI), D46.3 (SDO), D46.4 (SDI), D47.3 (SDO), D47.4 (SDI), D48.3 (SDO), D48.4 (SDI), D49.3 (SDO), D49.4 (SDI), D50.3 (SDO), D50.4 (SDI), D51.3 (SDO), D51.4 (SDI), D52.3 (SDO), D52.4 (SDI), D53.3 (SDO), D53.4 (SDI), D54.3 (SDO), D54.4 (SDI)
- net LED_DATA_unbuffered: now also U60.19 (IO11); no longer U60.18 (IO10)
- net MISO: now also IC5.7 (B4), U30.3 (MISO), U31.3 (MISO), U32.3 (MISO), U33.3 (MISO), U34.3 (MISO), U36.3 (MISO), U37.3 (MISO), U38.3 (MISO), U39.3 (MISO), U41.3 (MISO), U42.3 (MISO), U43.3 (MISO), U44.3 (MISO), U45.3 (MISO), U46.3 (MISO), U47.3 (MISO), U48.3 (MISO), U49.3 (MISO), U50.3 (MISO), U51.3 (MISO), U52.3 (MISO), U53.3 (MISO), U54.3 (MISO), U55.3 (MISO), U56.3 (MISO), U57.3 (MISO)
- net MISO unbuffered: now also IC5.5 (A4Y)
- net MOSI: now also IC4.18 (DIN), IC5.10 (B1Y), U30.2 (MOSI), U31.2 (MOSI), U32.2 (MOSI), U33.2 (MOSI), U34.2 (MOSI), U36.2 (MOSI), U37.2 (MOSI), U38.2 (MOSI), U39.2 (MOSI), U41.2 (MOSI), U42.2 (MOSI), U43.2 (MOSI), U44.2 (MOSI), U45.2 (MOSI), U46.2 (MOSI), U47.2 (MOSI), U48.2 (MOSI), U49.2 (MOSI), U50.2 (MOSI), U51.2 (MOSI), U52.2 (MOSI), U53.2 (MOSI), U54.2 (MOSI), U55.2 (MOSI), U56.2 (MOSI), U57.2 (MOSI)
- net MOSI unbuffered: now also IC5.2 (A1)
- net QRE_VIBRO_OUT: now also U60.21 (IO13); no longer U60.20 (IO12)
- net USB_D+: now also C8.1, J1.3; no longer C62.1, J1.2
- net USB_D-: now also C62.1, J1.2; no longer C8.1, J1.3
- new net CS00: IC4.17 (~{SYNC})
- new net SS_1: IC4.32 (S24), U30.4 (~{CS})
- new net SS_10: IC4.11 (S2), U41.4 (~{CS})
- new net SS_11: IC4.10 (S3), U42.4 (~{CS})
- new net SS_12: IC4.9 (S4), U43.4 (~{CS})
- new net SS_13: IC4.8 (S5), U44.4 (~{CS})
- new net SS_14: IC4.7 (S6), U45.4 (~{CS})
- new net SS_15: IC4.6 (S7), U46.4 (~{CS})
- new net SS_16: IC4.5 (S8), U47.4 (~{CS})
- new net SS_17: IC4.4 (S9), U48.4 (~{CS})
- new net SS_18: IC4.3 (S10), U49.4 (~{CS})
- new net SS_19: IC4.2 (S11), U50.4 (~{CS})
- new net SS_2: IC4.31 (S23), U31.4 (~{CS})
- new net SS_20: IC4.1 (S12), U51.4 (~{CS})
- new net SS_21: IC4.48 (S13), U52.4 (~{CS})
- new net SS_22: IC4.47 (S14), U53.4 (~{CS})
- new net SS_23: IC4.46 (S15), U54.4 (~{CS})
- new net SS_24: IC4.45 (S16), U55.4 (~{CS})
- new net SS_25: IC4.40 (S32), U56.4 (~{CS})
- new net SS_26: IC4.39 (S31), U57.4 (~{CS})
- new net SS_27: IC4.38 (S30)
- new net SS_28: IC4.37 (S29)
- new net SS_29: IC4.33 (S25)
- new net SS_3: IC4.30 (S22), U32.4 (~{CS})
- new net SS_30: IC4.34 (S26)
- new net SS_31: IC4.35 (S27)
- new net SS_32: IC4.36 (S28)
- new net SS_4: IC4.29 (S21), U33.4 (~{CS})
- new net SS_5: IC4.28 (S20), U34.4 (~{CS})
- new net SS_6: IC4.27 (S19), U36.4 (~{CS})
- new net SS_7: IC4.26 (S18), U37.4 (~{CS})
- new net SS_8: IC4.25 (S17), U38.4 (~{CS})
- new net SS_9: IC4.12 (S1), U39.4 (~{CS})
Other:
- moved on the sheet: C1, C2, C3, C30, C31, C32, C33, C34, C35, C4, C5, C6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

Commit message: xgfbdbg
Parts:
- added H10, H7, H8, H9: MountingHole, MountingHole:MountingHole_3.2mm_M3_DIN965, symbol Mechanical:MountingHole
Connections:
- net CLK: no longer IC4.19 (SCLK), IC5.9 (B2Y), U30.1 (SCLK), U31.1 (SCLK), U32.1 (SCLK), U33.1 (SCLK), U34.1 (SCLK), U36.1 (SCLK), U37.1 (SCLK), U38.1 (SCLK), U39.1 (SCLK), U41.1 (SCLK), U42.1 (SCLK), U43.1 (SCLK), U44.1 (SCLK), U45.1 (SCLK), U46.1 (SCLK), U47.1 (SCLK), U48.1 (SCLK), U49.1 (SCLK), U50.1 (SCLK), U51.1 (SCLK), U52.1 (SCLK), U53.1 (SCLK), U54.1 (SCLK), U55.1 (SCLK), U56.1 (SCLK), U57.1 (SCLK)
- net CS1: no longer IC4.43 (D), IC5.8 (B3Y)
- net MISO: no longer IC5.7 (B4), U30.3 (MISO), U31.3 (MISO), U32.3 (MISO), U33.3 (MISO), U34.3 (MISO), U36.3 (MISO), U37.3 (MISO), U38.3 (MISO), U39.3 (MISO), U41.3 (MISO), U42.3 (MISO), U43.3 (MISO), U44.3 (MISO), U45.3 (MISO), U46.3 (MISO), U47.3 (MISO), U48.3 (MISO), U49.3 (MISO), U50.3 (MISO), U51.3 (MISO), U52.3 (MISO), U53.3 (MISO), U54.3 (MISO), U55.3 (MISO), U56.3 (MISO), U57.3 (MISO)
- net MOSI: no longer IC4.18 (DIN), IC5.10 (B1Y), U30.2 (MOSI), U31.2 (MOSI), U32.2 (MOSI), U33.2 (MOSI), U34.2 (MOSI), U36.2 (MOSI), U37.2 (MOSI), U38.2 (MOSI), U39.2 (MOSI), U41.2 (MOSI), U42.2 (MOSI), U43.2 (MOSI), U44.2 (MOSI), U45.2 (MOSI), U46.2 (MOSI), U47.2 (MOSI), U48.2 (MOSI), U49.2 (MOSI), U50.2 (MOSI), U51.2 (MOSI), U52.2 (MOSI), U53.2 (MOSI), U54.2 (MOSI), U55.2 (MOSI), U56.2 (MOSI), U57.2 (MOSI)
- new net _CLK: IC4.19 (SCLK), IC5.9 (B2Y), U30.1 (SCLK), U31.1 (SCLK), U32.1 (SCLK), U33.1 (SCLK), U34.1 (SCLK), U36.1 (SCLK), U37.1 (SCLK), U38.1 (SCLK), U39.1 (SCLK), U41.1 (SCLK), U42.1 (SCLK), U43.1 (SCLK), U44.1 (SCLK), U45.1 (SCLK), U46.1 (SCLK), U47.1 (SCLK), U48.1 (SCLK), U49.1 (SCLK), U50.1 (SCLK), U51.1 (SCLK), U52.1 (SCLK), U53.1 (SCLK), U54.1 (SCLK), U55.1 (SCLK), U56.1 (SCLK), U57.1 (SCLK)
- new net _CS1: IC4.43 (D), IC5.8 (B3Y)
- new net _MISO: IC5.7 (B4), U30.3 (MISO), U31.3 (MISO), U32.3 (MISO), U33.3 (MISO), U34.3 (MISO), U36.3 (MISO), U37.3 (MISO), U38.3 (MISO), U39.3 (MISO), U41.3 (MISO), U42.3 (MISO), U43.3 (MISO), U44.3 (MISO), U45.3 (MISO), U46.3 (MISO), U47.3 (MISO), U48.3 (MISO), U49.3 (MISO), U50.3 (MISO), U51.3 (MISO), U52.3 (MISO), U53.3 (MISO), U54.3 (MISO), U55.3 (MISO), U56.3 (MISO), U57.3 (MISO)
- new net _MOSI: IC4.18 (DIN), IC5.10 (B1Y), U30.2 (MOSI), U31.2 (MOSI), U32.2 (MOSI), U33.2 (MOSI), U34.2 (MOSI), U36.2 (MOSI), U37.2 (MOSI), U38.2 (MOSI), U39.2 (MOSI), U41.2 (MOSI), U42.2 (MOSI), U43.2 (MOSI), U44.2 (MOSI), U45.2 (MOSI), U46.2 (MOSI), U47.2 (MOSI), U48.2 (MOSI), U49.2 (MOSI), U50.2 (MOSI), U51.2 (MOSI), U52.2 (MOSI), U53.2 (MOSI), U54.2 (MOSI), U55.2 (MOSI), U56.2 (MOSI), U57.2 (MOSI)
Other:
- moved on the sheet: C3, C4, C7, H3, H4, H5, H6

Commit message: yoyoyoyoy
Parts:
- added R10, R11, R12, R13, R14, R15, R16, R17, R18, R19, R20, R21, R22, R23, R24, R25, R26, R27, R28, R29, R30, R31, R32, R33, R34, R35, R36, R37, R38, R39, R4, R40, R41, R42, R43, R44, R45, R46, R47, R48, R49, R5, R50, R51, R52, R53, R54, R55, R6, R7, R8, R9: 10k, Resistor_SMD:R_0402_1005Metric, symbol Device:R
- R1, R2: footprint Resistor_SMD:R_0402_1005Metric -> Resistor_SMD:R_0805_2012Metric_Pad1.20x1.40mm_HandSolder
- renumbered R12 to R60, R13 to R61, U36 to U35, U37 to U36, U38 to U37, U39 to U38, U41 to U39, U42 to U40, U43 to U41, U44 to U42, U45 to U43, U46 to U44, U47 to U45, U48 to U46, U49 to U47, U50 to U48, U51 to U49, U52 to U50, U53 to U51, U54 to U52, U55 to U53, U56 to U54, U57 to U55, U35 to U62
Connections:
- net CS00 is gone; now on net _MUX_SYNC: IC4.17 (~{SYNC})
- net 3.3V: now also R10.2, R11.2, R12.2, R13.2, R14.2, R15.2, R16.2, R17.2, R18.2, R19.2, R20.2, R21.2, R22.2, R23.2, R24.2, R25.2, R26.2, R27.2, R28.2, R29.2, R30.2, R31.2, R32.2, R33.2, R34.2, R35.2, R36.2, R37.2, R38.2, R39.2, R4.2, R40.2, R41.2, R42.2, R43.2, R44.2, R45.2, R46.2, R47.2, R48.2, R49.2, R5.2, R50.2, R51.2, R52.2, R53.2, R54.2, R55.2, R6.2, R7.2, R8.2, R9.2
- net SS1: now also R4.1
- net SS10: now also R13.1
- net SS11: now also R14.1
- net SS12: now also R15.1
- net SS13: now also R16.1
- net SS14: now also R17.1
- net SS15: now also R18.1
- net SS16: now also R19.1
- net SS17: now also R20.1
- net SS18: now also R21.1
- net SS19: now also R22.1
- net SS2: now also R5.1
- net SS20: now also R23.1
- net SS21: now also R24.1
- net SS22: now also R25.1
- net SS23: now also R26.1
- net SS24: now also R27.1
- net SS25: now also R28.1
- net SS26: now also R29.1
- net SS3: now also R6.1
- net SS4: now also R7.1
- net SS5: now also R8.1
- net SS6: now also R9.1
- net SS7: now also R10.1
- net SS8: now also R11.1
- net SS9: now also R12.1
- net SS_1: now also R30.1
- net SS_10: now also R39.1
- net SS_11: now also R40.1
- net SS_12: now also R41.1
- net SS_13: now also R42.1
- net SS_14: now also R43.1
- net SS_15: now also R44.1
- net SS_16: now also R45.1
- net SS_17: now also R46.1
- net SS_18: now also R47.1
- net SS_19: now also R48.1
- net SS_2: now also R31.1
- net SS_20: now also R49.1
- net SS_21: now also R50.1
- net SS_22: now also R51.1
- net SS_23: now also R52.1
- net SS_24: now also R53.1
- net SS_25: now also R54.1
- net SS_26: now also R55.1
- net SS_3: now also R32.1
- net SS_4: now also R33.1
- net SS_5: now also R34.1
- net SS_6: now also R35.1
- net SS_7: now also R36.1
- net SS_8: now also R37.1
- net SS_9: now also R38.1
- net _MUX_SYNC: now reaches U60.17 (IO9)
- net CS0 renamed MUX_SYNC
- net LDC_CLK: no longer names the net of U60.10 (IO17)

Commit message: fgvjbhkljdtzrj
Other:
- note added: "MOUNTING HOLES"
- note added: "REFLECTIVE IMPACT SENSOR"
- note added: "RIVET HOLES"
- note added: "SPI BUFFER AND MUX (left & right)"
- note added: "TMAG5170 MAGNETIC SENSOR ARRAY"
- note removed: "REFLECTIVE VIBROMETER"
- note removed: "SPI BUFFER AND MUX"
- moved on the sheet: C2, C3, C4, C6, C62, C63, C64, C65, C7, C8, C9, H1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

Commit message: before production / pinout ESP IO
Parts:
- added J35: Conn_01x01_Pin, Connector_PinSocket_1.00mm:PinSocket_1x11_P1.00mm_Vertical, symbol Connector:Conn_01x11_Pin
Connections:
- net IO35: now reaches U60.28 (IO35)
- net IO36: now reaches U60.29 (IO36)
- net IO36: now also J35.10 (Pin_10)
- net IO37: now reaches U60.30 (IO37)
- net IO37: now also J35.9 (Pin_9)
- net IO38: now reaches U60.31 (IO38)
- net IO38: now also J35.8 (Pin_8)
- net IO39: now reaches U60.32 (IO39)
- net IO39: now also J35.7 (Pin_7)
- net IO40: now reaches U60.33 (IO40)
- net IO40: now also J35.6 (Pin_6)
- net IO41: now reaches U60.34 (IO41)
- net IO41: now also J35.5 (Pin_5)
- net IO42: now reaches U60.35 (IO42)
- net IO42: now also J35.4 (Pin_4)
- net RXD0: now reaches U60.36 (RXD0)
- net RXD0: now also J35.3 (Pin_3)
- net TXD0: now reaches U60.37 (TXD0)
- net TXD0: now also J35.2 (Pin_2)
- net Motor_PWM: now reaches U60.38 (IO2)
- net Motor_PWM: now also J35.11 (Pin_11)
- new net IO02: J35.1 (Pin_1)
