File: percussiveInterface-3.2/main_board_4_jlc/main_board_4_jlc-3.2.kicad_sch (KiCad schematic)
At the start: 83 parts, among them IC1 ADG731BSUZ, IC2 TXU0304RUTR, IC3 LM3940IMP-3.3_NOPB, J1 0022232041, J10 SAMTEC-SLW-108-01-X-S, J11 Screw_Terminal_01x02, J5 SLW-104-01-G-S, J6 SLW-104-01-G-S, J7 SLW-104-01-G-S, J8 SLW-104-01-G-S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

Commit message: asgfebgsdfbas
Parts:
- removed D1: APA102-2020, LED_SMD:LED-APA102-2020, symbol LED:APA102-2020
- added D12: LED_BGAR, LED_THT:LED_D5.0mm-4_RGB, symbol Device:LED_RAGB
- added R12: 220, Resistor_SMD:R_0402_1005Metric, symbol Device:R
- added R13: 100, Resistor_SMD:R_0402_1005Metric, symbol Device:R
- added R14: 200, Resistor_SMD:R_0402_1005Metric, symbol Device:R
Connections:
- net 5V: now also D12.2 (A)
- net LED_RED: now reaches U34.19 (IO11)
- net LED_RED: now also R14.1
- net LED_GREEN: now reaches U34.20 (IO12)
- net LED_GREEN: now also R13.1
- net LED_BLUE: now reaches U34.21 (IO13)
- net LED_BLUE: now also R12.1
- new net: D12.4 (BK), R12.2
- new net: D12.1 (RK), R14.2
- new net: D12.3 (GK), R13.2
